File: draft1/tutorial1/tutorial1.sch (KiCad schematic (older format))
At the start: 2 parts

Commit message: step 24
Parts:
- added D?: LED, symbol Device:LED
- added U?: PIC12C508A-ISM, Package_DIP:DIP-8_W7.62mm, symbol microchip_pic12mcu:PIC12C508A-ISM
Other:
- moved on the sheet: R?
Changed lines of the file:
@@
 L Device:R R?
 U 1 1 5ED6751A
-P 5500 4150
-F 0 "R?" V 5293 4150 50  0000 C CNN
-F 1 "1 k" V 5384 4150 50  0000 C CNN
-F 2 "" V 5430 4150 50  0001 C CNN
-F 3 "~" H 5500 4150 50  0001 C CNN
-	1    5500 4150
+P 6200 3050
+F 0 "R?" V 5993 3050 50  0000 C CNN
+F 1 "1 k" V 6084 3050 50  0000 C CNN
+F 2 "" V 6130 3050 50  0001 C CNN
+F 3 "~" H 6200 3050 50  0001 C CNN
+	1    6200 3050
 	0    1    1    0
 $EndComp
@@
 L Device:R R?
 U 1 1 5ED684D0
-P 6900 3750
-F 0 "R?" V 7107 3750 50  0000 C CNN
-F 1 "100" V 7016 3750 50  0000 C CNN
-F 2 "" V 6830 3750 50  0001 C CNN
-F 3 "~" H 6900 3750 50  0001 C CNN
-	1    6900 3750
+P 5600 4450
+F 0 "R?" V 5807 4450 50  0000 C CNN
+F 1 "100" V 5716 4450 50  0000 C CNN
+F 2 "" V 5530 4450 50  0001 C CNN
+F 3 "~" H 5600 4450 50  0001 C CNN
+	1    5600 4450
 	0    -1   -1   0
 $EndComp
+$Comp
+L microchip_pic12mcu:PIC12C508A-ISM U?
+U 1 1 5ED74B91
+P 3500 3800
+F 0 "U?" H 3500 4581 50  0000 C CNN
+F 1 "PIC12C508A-ISM" H 3500 4490 50  0000 C CNN
+F 2 "Package_DIP:DIP-8_W7.62mm" H 4100 4450 50  0001 C CNN
+F 3 "http://ww1.microchip.com/downloads/en/devicedoc/40139e.pdf" H 3500 3800 50  0001 C CNN
+	1    3500 3800
+	-1   0    0    -1
+$EndComp
+$Comp
+L Device:LED D?
+U 1 1 5ED76AD6
+P 5650 3050
+F 0 "D?" H 5643 3267 50  0000 C CNN
+F 1 "LED" H 5643 3176 50  0000 C CNN
+F 2 "" H 5650 3050 50  0001 C CNN
+F 3 "~" H 5650 3050 50  0001 C CNN
+	1    5650 3050
+	1    0    0    -1
+$EndComp
 $EndSCHEMATC

Commit message: step 48
Parts:
- added J1: MYCONN3, symbol microchip_pic12mcu:MYCONN3
- gave numbers to parts that had none: 4
Connections:
- net VCC: now reaches R2.1
- net VCC: now also U1.1 (VDD), J1.1 (VCC)
- net LEDtoR: now reaches R2.2
- net LEDtoR: now also D1.2 (A)
- net INPUTtoR: now reaches R1.1
- net INPUTtoR: now also J1.2 (INPUT)
- net INPUT: now reaches R1.2
- net INPUT: now also U1.6 (GP1)
- net uCtoLED: now reaches U1.7 (GP0)
- net uCtoLED: now also D1.1 (K)
- net GND: now reaches U1.8 (VSS)
- net GND: now also J1.3 (GND)
- no-connect marks 0 -> 4
Other:
- note added: "might not have attached these right"
- moved on the sheet: R1
Changed lines of the file:
@@
 $EndDescr
 $Comp
-L Device:R R?
+L Device:R R2
 U 1 1 5ED6751A
 P 6200 3050
-F 0 "R?" V 5993 3050 50  0000 C CNN
+F 0 "R2" V 5993 3050 50  0000 C CNN
 F 1 "1 k" V 6084 3050 50  0000 C CNN
 F 2 "" V 6130 3050 50  0001 C CNN
@@
 $EndComp
 $Comp
-L Device:R R?
+L Device:R R1
 U 1 1 5ED684D0
-P 5600 4450
-F 0 "R?" V 5807 4450 50  0000 C CNN
-F 1 "100" V 5716 4450 50  0000 C CNN
-F 2 "" V 5530 4450 50  0001 C CNN
-F 3 "~" H 5600 4450 50  0001 C CNN
-	1    5600 4450
+P 5550 5600
+F 0 "R1" V 5757 5600 50  0000 C CNN
+F 1 "100" V 5666 5600 50  0000 C CNN
+F 2 "" V 5480 5600 50  0001 C CNN
+F 3 "~" H 5550 5600 50  0001 C CNN
+	1    5550 5600
 	0    -1   -1   0
 $EndComp
 $Comp
-L microchip_pic12mcu:PIC12C508A-ISM U?
+L microchip_pic12mcu:PIC12C508A-ISM U1
 U 1 1 5ED74B91
 P 3500 3800
-F 0 "U?" H 3500 4581 50  0000 C CNN
-F 1 "PIC12C508A-ISM" H 3500 4490 50  0000 C CNN
+F 0 "U1" H 3200 4600 50  0000 C CNN
+F 1 "PIC12C508A-ISM" H 3100 4500 50  0000 C CNN
 F 2 "Package_DIP:DIP-8_W7.62mm" H 4100 4450 50  0001 C CNN
 F 3 "http://ww1.microchip.com/downloads/en/devicedoc/40139e.pdf" H 3500 3800 50  0001 C CNN
@@
 $EndComp
 $Comp
-L Device:LED D?
+L Device:LED D1
 U 1 1 5ED76AD6
 P 5650 3050
-F 0 "D?" H 5643 3267 50  0000 C CNN
+F 0 "D1" H 5643 3267 50  0000 C CNN
 F 1 "LED" H 5643 3176 50  0000 C CNN
 F 2 "" H 5650 3050 50  0001 C CNN
@@
 	1    0    0    -1
 $EndComp
+$Comp
+L microchip_pic12mcu:MYCONN3 J1
+U 1 1 5EDA0556
+P 3950 5400
+F 0 "J1" H 3700 5000 50  0000 C CNN
+F 1 "MYCONN3" H 3733 5434 50  0000 C CNN
+F 2 "" H 3950 5400 50  0001 C CNN
+F 3 "" H 3950 5400 50  0001 C CNN
+	1    3950 5400
+	1    0    0    -1
+$EndComp
+$Comp
+L power:VCC #PWR05
+U 1 1 5EDB0595
+P 6450 2950
+F 0 "#PWR05" H 6450 2800 50  0001 C CNN
+F 1 "VCC" H 6465 3123 50  0000 C CNN
+F 2 "" H 6450 2950 50  0001 C CNN
+F 3 "" H 6450 2950 50  0001 C CNN
+	1    6450 2950
+	1    0    0    -1
+$EndComp
+$Comp
+L power:VCC #PWR01
+U 1 1 5EDB2DA0
+P 3500 2900
+F 0 "#PWR01" H 3500 2750 50  0001 C CNN
+F 1 "VCC" H 3515 3073 50  0000 C CNN
+F 2 "" H 3500 2900 50  0001 C CNN
+F 3 "" H 3500 2900 50  0001 C CNN
+	1    3500 2900
+	1    0    0    -1
+$EndComp
+$Comp
+L power:VCC #PWR03
+U 1 1 5EDB3B1A
+P 4100 5450
+F 0 "#PWR03" H 4100 5300 50  0001 C CNN
+F 1 "VCC" H 4115 5623 50  0000 C CNN
+F 2 "" H 4100 5450 50  0001 C CNN
+F 3 "" H 4100 5450 50  0001 C CNN
+	1    4100 5450
+	1    0    0    -1
+$EndComp
+$Comp
+L power:GND #PWR02
+U 1 1 5EDC9F18
+P 3500 4550
+F 0 "#PWR02" H 3500 4300 50  0001 C CNN
+F 1 "GND" H 3505 4377 50  0000 C CNN
+F 2 "" H 3500 4550 50  0001 C CNN
+F 3 "" H 3500 4550 50  0001 C CNN
+	1    3500 4550
+	1    0    0    -1
+$EndComp
+$Comp
+L power:GND #PWR04
+U 1 1 5EDCBA30
+P 4100 5850
+F 0 "#PWR04" H 4100 5600 50  0001 C CNN
+F 1 "GND" H 4105 5677 50  0000 C CNN
+F 2 "" H 4100 5850 50  0001 C CNN
+F 3 "" H 4100 5850 50  0001 C CNN
+	1    4100 5850
+	1    0    0    -1
+$EndComp
+Wire Wire Line
+	4100 3700 4850 3700
+Wire Wire Line
+	4850 3700 4850 3050
+Wire Wire Line
+	4850 3050 5500 3050
+Wire Wire Line
+	5800 3050 6050 3050
+Wire Wire Line
+	6350 3050 6450 3050
+Wire Wire Line
+	6450 3050 6450 2950
+Wire Wire Line
+	3500 4400 3500 4550
+Wire Wire Line
+	3500 2900 3500 3200
+Wire Wire Line
+	3950 5600 5400 5600
+Wire Wire Line
+	4100 5850 4100 5700
+Wire Wire Line
+	4100 5700 3950 5700
+Wire Wire Line
+	4100 5450 3950 5450
+Wire Wire Line
+	3950 5450 3950 5500
+Wire Wire Line
+	4100 3800 4850 3800
+Text Label 4850 3800 0    50   ~ 0
+INPUT
+Wire Wire Line
+	5700 5600 6400 5600
+Text Label 6400 5600 0    50   ~ 0
+INPUT
+Text Label 4850 3250 0    50   ~ 0
+uCtoLED
+Text Label 5800 3050 0    50   ~ 0
+LEDtoR
+Text Label 4850 5600 0    50   ~ 0
+INPUTtoR
+NoConn ~ 2900 3900
+NoConn ~ 2900 3800
+NoConn ~ 2900 3700
+NoConn ~ 4100 3900
+$Comp
+L power:PWR_FLAG #FLG01
+U 1 1 5EDD3B19
+P 7300 3950
+F 0 "#FLG01" H 7300 4025 50  0001 C CNN
+F 1 "PWR_FLAG" H 7300 4123 50  0000 C CNN
+F 2 "" H 7300 3950 50  0001 C CNN
+F 3 "~" H 7300 3950 50  0001 C CNN
+	1    7300 3950
+	1    0    0    -1
+$EndComp
+$Comp
+L power:PWR_FLAG #FLG02
+U 1 1 5EDD4F83
+P 7850 3900
+F 0 "#FLG02" H 7850 3975 50  0001 C CNN
+F 1 "PWR_FLAG" H 7850 4073 50  0000 C CNN
+F 2 "" H 7850 3900 50  0001 C CNN
+F 3 "~" H 7850 3900 50  0001 C CNN
+	1    7850 3900
+	1    0    0    -1
+$EndComp
+$Comp
+L power:GND #PWR06
+U 1 1 5EDD60BF
+P 7300 3950
+F 0 "#PWR06" H 7300 3700 50  0001 C CNN
+F 1 "GND" H 7305 3777 50  0000 C CNN
+F 2 "" H 7300 3950 50  0001 C CNN
+F 3 "" H 7300 3950 50  0001 C CNN
+	1    7300 3950
+	1    0    0    -1
+$EndComp
+$Comp
+L power:VCC #PWR07
+U 1 1 5EDD7261
+P 7850 3900
+F 0 "#PWR07" H 7850 3750 50  0001 C CNN
+F 1 "VCC" H 7865 4073 50  0000 C CNN
+F 2 "" H 7850 3900 50  0001 C CNN
+F 3 "" H 7850 3900 50  0001 C CNN
+	1    7850 3900
+	-1   0    0    1
+$EndComp
+Text Notes 7550 3550 0    50   ~ 0
+might not have attached these right
 $EndSCHEMATC

Commit message: step 22
Parts:
- D1: footprint (none) -> LED_THT:LED_D5.0mm
- J1: footprint (none) -> Connector:Banana_Jack_3Pin
- R1, R2: footprint (none) -> Resistor_THT:R_Axial_DIN0207_L6.3mm_D2.5mm_P2.54mm_Vertical
Changed lines of the file:
@@
 F 0 "R2" V 5993 3050 50  0000 C CNN
 F 1 "1 k" V 6084 3050 50  0000 C CNN
-F 2 "" V 6130 3050 50  0001 C CNN
+F 2 "Resistor_THT:R_Axial_DIN0207_L6.3mm_D2.5mm_P2.54mm_Vertical" V 6130 3050 50  0001 C CNN
 F 3 "~" H 6200 3050 50  0001 C CNN
 	1    6200 3050
@@
 F 0 "R1" V 5757 5600 50  0000 C CNN
 F 1 "100" V 5666 5600 50  0000 C CNN
-F 2 "" V 5480 5600 50  0001 C CNN
+F 2 "Resistor_THT:R_Axial_DIN0207_L6.3mm_D2.5mm_P2.54mm_Vertical" V 5480 5600 50  0001 C CNN
 F 3 "~" H 5550 5600 50  0001 C CNN
 	1    5550 5600
@@
 F 0 "D1" H 5643 3267 50  0000 C CNN
 F 1 "LED" H 5643 3176 50  0000 C CNN
-F 2 "" H 5650 3050 50  0001 C CNN
+F 2 "LED_THT:LED_D5.0mm" H 5650 3050 50  0001 C CNN
 F 3 "~" H 5650 3050 50  0001 C CNN
 	1    5650 3050
@@
 F 0 "J1" H 3700 5000 50  0000 C CNN
 F 1 "MYCONN3" H 3733 5434 50  0000 C CNN
-F 2 "" H 3950 5400 50  0001 C CNN
+F 2 "Connector:Banana_Jack_3Pin" H 3950 5400 50  0001 C CNN
 F 3 "" H 3950 5400 50  0001 C CNN
 	1    3950 5400
