File: draft1/tutorial1/tutorial1.kicad_pcb (KiCad board)
At the start: 2 copper layers, 59.7 x 48.3 mm, 5 parts, among them J1 MYCONN3, U1 PIC12C508A-ISM

Commit message: autorouted
Routing:
- net GND: track 59.8 -> 0.00 mm, vias 2 -> 0
- net /INPUTtoR: track 38.6 -> 32.8 mm
- net VCC: track 39.5 -> 36.0 mm
- added copper zone on B.Cu, net GND
Other:
- board outline removed
Changed lines of the file:
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@@
   (general
     (thickness 1.6)
-    (drawings 4)
-    (tracks 28)
+    (drawings 0)
+    (tracks 15)
     (zones 0)
     (modules 5)
@@
     (visible_elements 7FFFFFFF)
     (pcbplotparams
-      (layerselection 0x010fc_ffffffff)
+      (layerselection 0x010f0_ffffffff)
       (usegerberextensions false)
       (usegerberattributes true)
@@
       (outputformat 1)
       (mirror false)
-      (drillshape 1)
+      (drillshape 0)
       (scaleselection 1)
-      (outputdirectory ""))
+      (outputdirectory "gerber files/"))
   )
   (net 0 "")
@@
     )
   )
-  (gr_line (start 176.53 85.09) (end 116.84 85.09) (layer Edge.Cuts) (width 0.05))
-  (gr_line (start 176.53 133.35) (end 176.53 85.09) (layer Edge.Cuts) (width 0.05))
-  (gr_line (start 116.84 133.35) (end 176.53 133.35) (layer Edge.Cuts) (width 0.05))
-  (gr_line (start 116.84 85.09) (end 116.84 133.35) (layer Edge.Cuts) (width 0.05))
-  (segment (start 127 113.03) (end 122.5 108.53) (width 0.6096) (layer F.Cu) (net 1))
-  (segment (start 122.5 95.83) (end 121.92 95.25) (width 0.6096) (layer F.Cu) (net 1))
-  (segment (start 122.5 108.53) (end 122.5 95.83) (width 0.6096) (layer F.Cu) (net 1))
-  (segment (start 142.901106 95.25) (end 147.981106 90.17) (width 0.6096) (layer F.Cu) (net 2))
-  (segment (start 147.981106 90.17) (end 148.59 90.17) (width 0.6096) (layer F.Cu) (net 2))
-  (segment (start 124.46 95.25) (end 142.901106 95.25) (width 0.6096) (layer F.Cu) (net 2))
-  (segment (start 166.37 99.06) (end 166.37 106.13) (width 0.6096) (layer F.Cu) (net 3))
-  (segment (start 166.37 106.13) (end 162.5 110) (width 0.6096) (layer F.Cu) (net 3))
-  (segment (start 162.5 110) (end 152.5 110) (width 0.6096) (layer F.Cu) (net 3))
-  (segment (start 148.59 113.91) (end 148.59 124.46) (width 0.6096) (layer F.Cu) (net 3))
-  (segment (start 152.5 110) (end 148.59 113.91) (width 0.6096) (layer F.Cu) (net 3))
-  (segment (start 163.57 124.46) (end 151.61 112.5) (width 0.6096) (layer B.Cu) (net 4))
-  (segment (start 151.61 112.5) (end 142.5 112.5) (width 0.6096) (layer B.Cu) (net 4))
-  (segment (start 142.5 112.5) (end 135 105) (width 0.6096) (layer B.Cu) (net 4))
-  (segment (start 135 105) (end 135 95) (width 0.6096) (layer B.Cu) (net 4))
-  (via (at 137.5 92.5) (size 0.8) (drill 0.4) (layers F.Cu B.Cu) (net 4))
-  (segment (start 135 95) (end 137.5 92.5) (width 0.6096) (layer B.Cu) (net 4))
-  (via (at 140 90) (size 0.8) (drill 0.4) (layers F.Cu B.Cu) (net 4))
-  (segment (start 137.5 92.5) (end 140 90) (width 0.6096) (layer F.Cu) (net 4))
-  (segment (start 145.88 90) (end 146.05 90.17) (width 0.6096) (layer B.Cu) (net 4))
-  (segment (start 140 90) (end 145.88 90) (width 0.6096) (layer B.Cu) (net 4))
+  (segment (start 127 113.03) (end 127 111.7249) (width 0.6096) (layer B.Cu) (net 1))
+  (segment (start 121.92 95.25) (end 121.92 106.6449) (width 0.6096) (layer B.Cu) (net 1))
+  (segment (start 121.92 106.6449) (end 127 111.7249) (width 0.6096) (layer B.Cu) (net 1))
+  (segment (start 124.46 95.25) (end 142.901 95.25) (width 0.6096) (layer F.Cu) (net 2))
+  (segment (start 142.901 95.25) (end 147.981 90.17) (width 0.6096) (layer F.Cu) (net 2))
+  (segment (start 147.981 90.17) (end 148.59 90.17) (width 0.6096) (layer F.Cu) (net 2))
+  (segment (start 148.59 124.46) (end 166.37 106.68) (width 0.6096) (layer B.Cu) (net 3))
+  (segment (start 166.37 106.68) (end 166.37 99.06) (width 0.6096) (layer B.Cu) (net 3))
+  (segment (start 146.05 97.79) (end 144.7449 97.79) (width 0.6096) (layer B.Cu) (net 5))
+  (segment (start 129.54 113.03) (end 144.7449 97.8251) (width 0.6096) (layer B.Cu) (net 5))
+  (segment (start 144.7449 97.8251) (end 144.7449 97.79) (width 0.6096) (layer B.Cu) (net 5))
+  (segment (start 133.6 124.46) (end 133.6 117.09) (width 0.6096) (layer F.Cu) (net 5))
   (segment (start 133.6 117.09) (end 129.54 113.03) (width 0.6096) (layer F.Cu) (net 5))
-  (segment (start 133.6 124.46) (end 133.6 117.09) (width 0.6096) (layer F.Cu) (net 5))
-  (segment (start 146.05 103.95) (end 146.05 97.79) (width 0.6096) (layer F.Cu) (net 5))
-  (segment (start 129.54 113.03) (end 136.97 113.03) (width 0.6096) (layer F.Cu) (net 5))
-  (segment (start 136.97 113.03) (end 146.05 103.95) (width 0.6096) (layer F.Cu) (net 5))
-  (segment (start 157.48 96.52) (end 166.37 96.52) (width 0.6096) (layer F.Cu) (net 6))
-  (segment (start 151.13 90.17) (end 157.48 96.52) (width 0.6096) (layer F.Cu) (net 6))
+  (segment (start 166.37 96.52) (end 157.48 96.52) (width 0.6096) (layer F.Cu) (net 6))
+  (segment (start 157.48 96.52) (end 151.13 90.17) (width 0.6096) (layer F.Cu) (net 6))
+  (zone (net 4) (net_name GND) (layer B.Cu) (hatch edge 0.508)
+    (connect_pads (clearance 0.508))
+    (min_thickness 0.254)
+    (fill yes (arc_segments 32) (thermal_gap 0.508) (thermal_bridge_width 0.508))
+    (polygon
+      (pts
+        (xy 173.5836 135.9408) (xy 107.95 135.9408) (xy 107.95 84.1756) (xy 173.5836 84.1756)
+      )
+    )
+  )
 )
