File: scum3c_devboard/scan_chain_boot.sch (KiCad schematic (older format))
At the start: 5 parts, among them P4 Conn_01x24, U5 74AVC4TD245PW,118, U6 74AVC4TD245PW,118

Commit message: changed resistor smd footprint to 0402
Parts:
- R7, R8: footprint Resistor_SMD:R_0603_1608Metric -> Resistor_SMD:R_0402_1005Metric
Changed lines of the file:
@@
 F 0 "R7" V 3845 3250 50  0000 C CNN
 F 1 "NP" V 3936 3250 50  0000 C CNN
-F 2 "Resistor_SMD:R_0603_1608Metric" V 4090 3240 50  0001 C CNN
+F 2 "Resistor_SMD:R_0402_1005Metric" V 4090 3240 50  0001 C CNN
 F 3 "~" H 4050 3250 50  0001 C CNN
 	1    4050 3250
@@
 F 0 "R8" V 4795 2150 50  0000 C CNN
 F 1 "100k" V 4886 2150 50  0000 C CNN
-F 2 "Resistor_SMD:R_0603_1608Metric" V 5040 2140 50  0001 C CNN
+F 2 "Resistor_SMD:R_0402_1005Metric" V 5040 2140 50  0001 C CNN
 F 3 "~" H 5000 2150 50  0001 C CNN
 	1    5000 2150
