File: scum3c_devboard/scum3c-devboard.sch (KiCad schematic (older format))
At the start: 10 parts, among them U10 LTC4123, U9AB1 MPU-9250

Commit message: changed resistor smd footprint to 0402
Parts:
- R9: footprint Resistor_SMD:R_0603_1608Metric -> Resistor_SMD:R_0402_1005Metric
Changed lines of the file:
@@
 F 0 "R9" H 5468 4646 50  0000 L CNN
 F 1 "NP" H 5468 4555 50  0000 L CNN
-F 2 "Resistor_SMD:R_0603_1608Metric" V 5440 4590 50  0001 C CNN
+F 2 "Resistor_SMD:R_0402_1005Metric" V 5440 4590 50  0001 C CNN
 F 3 "~" H 5400 4600 50  0001 C CNN
 	1    5400 4600
