File: scum3c_devboard/uart.sch (KiCad schematic (older format))
At the start: 25 parts, among them J1 47346-0001, P3 Conn_01x02, U1 LP5907MFX-1.5, U2 74AVC1T45GS,132, U3 FT231XS-U, U4 74AVC1T45GS,132

Commit message: changed resistor smd footprint to 0402
Parts:
- R1, R2, R3, R4, R5, R6: footprint Resistor_SMD:R_0603_1608Metric -> Resistor_SMD:R_0402_1005Metric
Changed lines of the file:
@@
 F 0 "R6" H 5682 4554 50  0000 R CNN
 F 1 "27" H 5682 4645 50  0000 R CNN
-F 2 "Resistor_SMD:R_0603_1608Metric" V 5790 4590 50  0001 C CNN
+F 2 "Resistor_SMD:R_0402_1005Metric" V 5790 4590 50  0001 C CNN
 F 3 "~" H 5750 4600 50  0001 C CNN
 	1    5750 4600
@@
 F 0 "R3" H 6168 4546 50  0000 L CNN
 F 1 "27" H 6168 4455 50  0000 L CNN
-F 2 "Resistor_SMD:R_0603_1608Metric" V 6140 4490 50  0001 C CNN
+F 2 "Resistor_SMD:R_0402_1005Metric" V 6140 4490 50  0001 C CNN
 F 3 "~" H 6100 4500 50  0001 C CNN
 	1    6100 4500
@@
 F 0 "R4" H 6418 3346 50  0000 L CNN
 F 1 "270" H 6418 3255 50  0000 L CNN
-F 2 "Resistor_SMD:R_0603_1608Metric" V 6390 3290 50  0001 C CNN
+F 2 "Resistor_SMD:R_0402_1005Metric" V 6390 3290 50  0001 C CNN
 F 3 "~" H 6350 3300 50  0001 C CNN
 	1    6350 3300
@@
 F 0 "R5" H 4068 4646 50  0000 L CNN
 F 1 "270" H 4068 4555 50  0000 L CNN
-F 2 "Resistor_SMD:R_0603_1608Metric" V 4040 4590 50  0001 C CNN
+F 2 "Resistor_SMD:R_0402_1005Metric" V 4040 4590 50  0001 C CNN
 F 3 "~" H 4000 4600 50  0001 C CNN
 	1    4000 4600
@@
 F 0 "R1" V 9905 1200 50  0000 C CNN
 F 1 "NP" V 9814 1200 50  0000 C CNN
-F 2 "Resistor_SMD:R_0603_1608Metric" V 9740 1190 50  0001 C CNN
+F 2 "Resistor_SMD:R_0402_1005Metric" V 9740 1190 50  0001 C CNN
 F 3 "~" H 9700 1200 50  0001 C CNN
 	1    9700 1200
@@
 F 0 "R2" V 9905 1650 50  0000 C CNN
 F 1 "NP" V 9814 1650 50  0000 C CNN
-F 2 "Resistor_SMD:R_0603_1608Metric" V 9740 1640 50  0001 C CNN
+F 2 "Resistor_SMD:R_0402_1005Metric" V 9740 1640 50  0001 C CNN
 F 3 "~" H 9700 1650 50  0001 C CNN
 	1    9700 1650
