File: scum3c_devboard_large/Teensy Conn.sch (KiCad schematic (older format))
At the start: 5 parts, among them J4 Conn_01x22, U10 74AVCH4T245D,118, U11 74AVCH4T245D,118, U13 74AVCH4T245D,118, U9 74AVCH4T245D,118

Commit message: Suggested changes
Parts:
- J4: footprint Connector_PinHeader_2.54mm:PinHeader_1x22_P2.54mm_Vertical -> SCUM:Teensy_Connector; symbol Connector_Generic:Conn_01x22 -> SCUM:Teensy_Connector
Connections:
- net +TEENSY33: now also J4.3.3V; no longer J4.1 (Pin_1)
- net 3WB_CLK33: now also J4.A2; no longer J4.9 (Pin_9)
- net 3WB_DATA33: now also J4.A0; no longer J4.11 (Pin_11)
- net 3WB_ENB33: now also J4.A1; no longer J4.10 (Pin_10)
- net Clock33: now also J4.A6; no longer J4.5 (Pin_5)
- net GND: now also J4.GND; no longer J4.13 (Pin_13)
- net GPIO0: now also J4.D13; no longer J4.12 (Pin_12)
- net GPIO1: now also J4.A7; no longer J4.4 (Pin_4)
- net GPIO2: now also J4.A5; no longer J4.6 (Pin_6)
- net GPIO3: now also J4.A20; no longer J4.16 (Pin_16)
- net RsRx: now also J4.RX5; no longer J4.21 (Pin_21)
- net RsTx: now also J4.TX5; no longer J4.22 (Pin_22)
- net aLOAD33: now also J4.A16; no longer J4.20 (Pin_20)
- net aPHI33: now also J4.A18; no longer J4.18 (Pin_18)
- net aPHIb33: now also J4.A19; no longer J4.17 (Pin_17)
- net aSCANIN33: now also J4.A8; no longer J4.3 (Pin_3)
- net aSCANOUT33: now also J4.A17; no longer J4.19 (Pin_19)
- net aSCSEL33: now also J4.A9; no longer J4.2 (Pin_2)
- net hReset33: now also J4.A3; no longer J4.8 (Pin_8)
- net sReset33: now also J4.A4; no longer J4.7 (Pin_7)
Changed lines of the file:
@@
 EESchema Schematic File Version 4
 LIBS:scum3c-devboard-cache
-EELAYER 26 0
+EELAYER 30 0
 EELAYER END
 $Descr A4 11693 8268
 encoding utf-8
-Sheet 4 4
+Sheet 3 4
 Title ""
 Date ""
@@
 $EndDescr
 $Comp
-L Connector_Generic:Conn_01x22 J?
+L SCUM:Teensy_Connector J?
 U 1 1 5FCB6CAE
 P 1400 1950
@@
 F 0 "J4" H 1480 1942 50  0000 L CNN
 F 1 "Conn_01x22" H 1480 1851 50  0000 L CNN
-F 2 "Connector_PinHeader_2.54mm:PinHeader_1x22_P2.54mm_Vertical" H 1400 1950 50  0001 C CNN
+F 2 "SCUM:Teensy_Connector" H 1400 1950 50  0001 C CNN
 F 3 "~" H 1400 1950 50  0001 C CNN
 	1    1400 1950
@@
 $EndComp
 $Comp
-L draft1library:+VBAT #PWR0118
+L SCUM:+VBAT #PWR0118
 U 1 1 5FCB6DF9
 P 1050 3500
@@
 $EndComp
 $Comp
-L draft1library:+VBAT #PWR0142
+L SCUM:+VBAT #PWR0142
 U 1 1 5FCB6E2B
 P 1050 4600
@@
 Level Shifters
 $Comp
-L draft1library:+VBAT #PWR0166
+L SCUM:+VBAT #PWR0166
 U 1 1 6008365C
 P 1050 5700
@@
 sReset33
 $Comp
-L draft1library:+TEENSY33 #PWR0155
+L SCUM:+TEENSY33 #PWR0155
 U 1 1 6009E0D6
 P 1600 2950
@@
 $EndComp
 $Comp
-L draft1library:+VIN #PWR0159
+L SCUM:+VIN #PWR0159
 U 1 1 6009F474
 P 2350 3500
@@
 $EndComp
 $Comp
-L draft1library:+VIN #PWR0163
+L SCUM:+VIN #PWR0163
 U 1 1 6009F4B7
 P 2350 4600
@@
 $EndComp
 $Comp
-L draft1library:+VIN #PWR0164
+L SCUM:+VIN #PWR0164
 U 1 1 6009F4E5
 P 2350 5700
@@
 $EndComp
 $Comp
-L draft1library:+VBAT #PWR0192
+L SCUM:+VBAT #PWR0192
 U 1 1 600C6A13
 P 1050 6800
@@
 $EndComp
 $Comp
-L draft1library:+VIN #PWR0202
+L SCUM:+VIN #PWR0202
 U 1 1 600C6A35
 P 2350 6800
@@
 	2900 3300 2900 7700
 $Comp
-L draft1library:+VBAT #PWR0205
+L SCUM:+VBAT #PWR0205
 U 1 1 600C710E
 P 1050 6900

Commit message: switching computers
Parts:
- removed J4: Conn_01x22, SCUM:Teensy_Connector, symbol SCUM:Teensy_Connector
- added J6: Conn_01x24, Connector_PinSocket_2.54mm:PinSocket_1x24_P2.54mm_Vertical, symbol Connector_Generic:Conn_01x24
- U10, U11, U13, U9: symbol 74AVCH4T245D_118:74AVCH4T245D,118 -> SCUM:74AVCH4T245D,118
Connections:
- net +TEENSY33: now also J6.3 (Pin_3)
- net 3WB_CLK33: now also J6.8 (Pin_8)
- net 3WB_DATA33: now also J6.10 (Pin_10)
- net 3WB_ENB33: now also J6.9 (Pin_9)
- net Clock33: now also J6.13 (Pin_13)
- net GND: now also J6.15 (Pin_15), J6.6 (Pin_6)
- net GPIO0: now also J6.11 (Pin_11)
- net RsRx: now also J6.23 (Pin_23), J6.5 (Pin_5)
- net RsTx: now also J6.24 (Pin_24), J6.4 (Pin_4)
- net aLOAD33: now also J6.19 (Pin_19)
- net aPHI33: now also J6.18 (Pin_18)
- net aPHIb33: now also J6.14 (Pin_14)
- net aSCANIN33: now also J6.20 (Pin_20)
- net aSCANOUT33: now also J6.16 (Pin_16), J6.21 (Pin_21)
- net aSCSEL33: now also J6.17 (Pin_17), J6.22 (Pin_22)
- net hReset33: now also J6.7 (Pin_7)
- net sReset renamed GPO_ZERO
- net sReset33 renamed GPO_ZERO33
- net GPO_ZERO33: now also J6.12 (Pin_12)
Other:
- note added: "Teensy/nRF Connector"
- note removed: "Teensy"
Changed lines of the file:
@@
 $EndDescr
-$Comp
-L SCUM:Teensy_Connector J?
-U 1 1 5FCB6CAE
-P 1400 1950
-AR Path="/5FCB6CAE" Ref="J?"  Part="1"
-AR Path="/5FCB6A87/5FCB6CAE" Ref="J4"  Part="1"
-F 0 "J4" H 1480 1942 50  0000 L CNN
-F 1 "Conn_01x22" H 1480 1851 50  0000 L CNN
-F 2 "SCUM:Teensy_Connector" H 1400 1950 50  0001 C CNN
-F 3 "~" H 1400 1950 50  0001 C CNN
-	1    1400 1950
-	-1   0    0    1
-$EndComp
 $Comp
 L SCUM:+VBAT #PWR0118
@@
 L power:GND #PWR?
 U 1 1 5FCB782F
-P 1600 1750
+P 1800 1600
 AR Path="/5F3B307E/5FCB782F" Ref="#PWR?"  Part="1"
 AR Path="/5FCB782F" Ref="#PWR?"  Part="1"
 AR Path="/5FCB6A87/5FCB782F" Ref="#PWR0162"  Part="1"
-F 0 "#PWR0162" H 1600 1500 50  0001 C CNN
-F 1 "GND" V 1600 1650 50  0000 R CNN
-F 2 "" H 1600 1750 50  0001 C CNN
-F 3 "" H 1600 1750 50  0001 C CNN
-	1    1600 1750
-	0    -1   -1   0
-$EndComp
-NoConn ~ 1600 1650
-NoConn ~ 1600 1550
+F 0 "#PWR0162" H 1800 1350 50  0001 C CNN
+F 1 "GND" V 1800 1500 50  0000 R CNN
+F 2 "" H 1800 1600 50  0001 C CNN
+F 3 "" H 1800 1600 50  0001 C CNN
+	1    1800 1600
+	0    -1   -1   0
+$EndComp
 Text HLabel 1050 4000 0    50   Input ~ 0
 aSCANIN
 Text HLabel 1050 4100 0    50   Input ~ 0
 aSCSEL
-Text HLabel 1600 2650 2    50   Input ~ 0
-GPIO1
 Text HLabel 1050 4900 0    50   Input ~ 0
 Clock
-Text HLabel 1600 2450 2    50   Input ~ 0
-GPIO2
 Text HLabel 1050 6000 0    50   Input ~ 0
-sReset
+GPO_ZERO
 Text HLabel 1050 6300 0    50   Input ~ 0
 hReset
@@
 Text HLabel 1050 5000 0    50   Input ~ 0
 3WB_DATA
-Text HLabel 1600 1850 2    50   Input ~ 0
+Text HLabel 1750 2050 2    50   Input ~ 0
 GPIO0
-Text HLabel 1600 1450 2    50   Input ~ 0
-GPIO3
 Text HLabel 1050 6200 0    50   Input ~ 0
 aPHIb
@@
 Text HLabel 1050 3900 0    50   Input ~ 0
 aLOAD
-Text HLabel 1600 950  2    50   Input ~ 0
+Text HLabel 1750 850  2    50   Input ~ 0
 RsRx
-Text HLabel 1600 850  2    50   Input ~ 0
+Text HLabel 1750 750  2    50   Input ~ 0
 RsTx
 Text Label 2350 7100 0    50   ~ 0
 aSCANOUT33
-Text Label 1600 1050 0    50   ~ 0
+Text Label 1750 1250 0    50   ~ 0
 aLOAD33
-Text Label 1600 1150 0    50   ~ 0
+Text Label 1750 1550 0    50   ~ 0
 aSCANOUT33
 Text Label 2350 3900 0    50   ~ 0
@@
 Text Label 2350 4100 0    50   ~ 0
 aSCSEL33
-Text Label 1600 2750 0    50   ~ 0
+Text Label 1750 1150 0    50   ~ 0
 aSCANIN33
-Text Label 1600 2850 0    50   ~ 0
+Text Label 1750 1450 0    50   ~ 0
 aSCSEL33
 Text Label 2350 6100 0    50   ~ 0
 aPHI33
-Text Label 1600 1250 0    50   ~ 0
+Text Label 1750 1350 0    50   ~ 0
 aPHI33
 Text Label 2350 6200 0    50   ~ 0
@@
 Text Label 2350 6300 0    50   ~ 0
 hReset33
-Text Label 1600 2250 0    50   ~ 0
+Text Label 1750 2450 0    50   ~ 0
 hReset33
-Text Label 1600 1350 0    50   ~ 0
+Text Label 1750 1750 0    50   ~ 0
 aPHIb33
-Text Label 1600 2550 0    50   ~ 0
+Text Label 1750 1850 0    50   ~ 0
 Clock33
 Wire Notes Line
-	600  3200 600  600
-Wire Notes Line
 	600  7700 2900 7700
 Wire Notes Line
 	2900 3300 600  3300
 Wire Notes Line
-	2900 600  2900 3200
-Wire Notes Line
-	600  600  2900 600
+	2900 550  600  550
 Wire Notes Line
 	600  3200 2900 3200
-Text Notes 2550 3150 0    50   ~ 0
-Teensy
+Text Notes 2000 3150 0    50   ~ 0
+Teensy/nRF Connector
 Text Notes 2300 7650 0    50   ~ 0
 Level Shifters
@@
 Text Label 2350 5000 0    50   ~ 0
 3WB_DATA33
-Text Label 1600 2150 0    50   ~ 0
+Text Label 1750 2350 0    50   ~ 0
 3WB_CLK33
-Text Label 1600 2050 0    50   ~ 0
+Text Label 1750 2250 0    50   ~ 0
 3WB_ENB33
-Text Label 1600 1950 0    50   ~ 0
+Text Label 1750 2150 0    50   ~ 0
 3WB_DATA33
 Text Label 2350 6000 0    50   ~ 0
-sReset33
-Text Label 1600 2350 0    50   ~ 0
-sReset33
+GPO_ZERO33
 $Comp
 L SCUM:+TEENSY33 #PWR0155
 U 1 1 6009E0D6
-P 1600 2950
-F 0 "#PWR0155" H 1600 2800 50  0001 C CNN
-F 1 "+TEENSY33" V 1615 3077 50  0000 L CNN
-F 2 "" H 1600 2950 50  0001 C CNN
-F 3 "" H 1600 2950 50  0001 C CNN
-	1    1600 2950
+P 1750 2850
+F 0 "#PWR0155" H 1750 2700 50  0001 C CNN
+F 1 "+TEENSY33" V 1765 2977 50  0000 L CNN
+F 2 "" H 1750 2850 50  0001 C CNN
+F 3 "" H 1750 2850 50  0001 C CNN
+	1    1750 2850
 	0    1    1    0
 $EndComp
@@
 $EndComp
 $Comp
-L 74AVCH4T245D_118:74AVCH4T245D,118 U9
+L SCUM:74AVCH4T245D,118 U9
 U 1 1 6009FAD9
 P 1700 3850
@@
 $EndComp
 $Comp
-L 74AVCH4T245D_118:74AVCH4T245D,118 U10
+L SCUM:74AVCH4T245D,118 U10
 U 1 1 600A041E
 P 1700 4950
@@
 $EndComp
 $Comp
-L 74AVCH4T245D_118:74AVCH4T245D,118 U11
+L SCUM:74AVCH4T245D,118 U11
 U 1 1 600A0446
 P 1700 6050
@@
 $EndComp
 $Comp
-L 74AVCH4T245D_118:74AVCH4T245D,118 U13
+L SCUM:74AVCH4T245D,118 U13
 U 1 1 600C6A3D
 P 1700 7150
@@
 NoConn ~ 2350 7200
 NoConn ~ 1050 7200
+$Comp
+L Connector_Generic:Conn_01x24 J6
+U 1 1 60B65C85
+P 1550 1950
+F 0 "J6" H 1850 1850 50  0000 C CNN
+F 1 "Conn_01x24" H 1850 1950 50  0000 C CNN
+F 2 "Connector_PinSocket_2.54mm:PinSocket_1x24_P2.54mm_Vertical" H 1550 1950 50  0001 C CNN
+F 3 "~" H 1550 1950 50  0001 C CNN
+	1    1550 1950
+	-1   0    0    1
+$EndComp
+Wire Notes Line
+	2900 550  2900 3200
+Wire Notes Line
+	600  550  600  3200
+NoConn ~ 1750 3050
+NoConn ~ 1750 2950
+Text HLabel 1750 2650 2    50   Input ~ 0
+RsRx
+Text HLabel 1750 2750 2    50   Input ~ 0
+RsTx
+$Comp
+L power:GND #PWR?
+U 1 1 60B82D3E
+P 1750 2550
+AR Path="/5F3B307E/60B82D3E" Ref="#PWR?"  Part="1"
+AR Path="/60B82D3E" Ref="#PWR?"  Part="1"
+AR Path="/5FCB6A87/60B82D3E" Ref="#PWR0237"  Part="1"
+F 0 "#PWR0237" H 1750 2300 50  0001 C CNN
+F 1 "GND" V 1750 2450 50  0000 R CNN
+F 2 "" H 1750 2550 50  0001 C CNN
+F 3 "" H 1750 2550 50  0001 C CNN
+	1    1750 2550
+	0    -1   -1   0
+$EndComp
+Text Label 1750 1050 0    50   ~ 0
+aSCANOUT33
+Text Label 1750 950  0    50   ~ 0
+aSCSEL33
+Text Label 1750 1950 0    50   ~ 0
+GPO_ZERO33
+Wire Wire Line
+	1800 1600 1800 1650
+Wire Wire Line
+	1800 1650 1750 1650
 $EndSCHEMATC

Commit message: ready for review
Connections:
- net 3WB_CLK: now also U11.6 (2A1); no longer U10.7 (2A2)
- net 3WB_CLK33: now also U11.11 (2B1); no longer U10.10 (2B2)
- net 3WB_DATA: now also U11.4 (1A1); no longer U10.5 (1A2)
- net 3WB_DATA33: now also U11.13 (1B1); no longer U10.12 (1B2)
- net 3WB_ENB: now also U11.5 (1A2); no longer U10.6 (2A1)
- net 3WB_ENB33: now also U11.12 (1B2); no longer U10.11 (2B1)
- net Clock: now also U10.6 (2A1); no longer U10.4 (1A1)
- net Clock33: now also U10.11 (2B1); no longer U10.13 (1B1)
- net GPO_ZERO: now also U10.7 (2A2); no longer U11.4 (1A1)
- net GPO_ZERO33: now also U10.10 (2B2); no longer U11.13 (1B1)
- net aPHI: now also U9.6 (2A1); no longer U11.5 (1A2)
- net aPHI33: now also U9.11 (2B1); no longer U11.12 (1B2)
- net aPHIb: now also U10.5 (1A2); no longer U11.6 (2A1)
- net aPHIb33: now also U10.12 (1B2); no longer U11.11 (2B1)
- net aSCANIN: now also U9.4 (1A1); no longer U9.6 (2A1)
- net aSCANIN33: now also U9.13 (1B1); no longer U9.11 (2B1)
Changed lines of the file:
@@
 EESchema Schematic File Version 4
 LIBS:scum3c-devboard-cache
-EELAYER 30 0
+EELAYER 26 0
 EELAYER END
 $Descr A4 11693 8268
@@
 	0    -1   -1   0
 $EndComp
-Text HLabel 1050 4000 0    50   Input ~ 0
+Text HLabel 1050 3800 0    50   Input ~ 0
 aSCANIN
 Text HLabel 1050 4100 0    50   Input ~ 0
 aSCSEL
-Text HLabel 1050 4900 0    50   Input ~ 0
+Text HLabel 1050 5100 0    50   Input ~ 0
 Clock
-Text HLabel 1050 6000 0    50   Input ~ 0
+Text HLabel 1050 5200 0    50   Input ~ 0
 GPO_ZERO
 Text HLabel 1050 6300 0    50   Input ~ 0
 hReset
-Text HLabel 1050 5200 0    50   Input ~ 0
+Text HLabel 1050 6200 0    50   Input ~ 0
 3WB_CLK
-Text HLabel 1050 5100 0    50   Input ~ 0
+Text HLabel 1050 6100 0    50   Input ~ 0
 3WB_ENB
-Text HLabel 1050 5000 0    50   Input ~ 0
+Text HLabel 1050 6000 0    50   Input ~ 0
 3WB_DATA
 Text HLabel 1750 2050 2    50   Input ~ 0
 GPIO0
-Text HLabel 1050 6200 0    50   Input ~ 0
+Text HLabel 1050 5000 0    50   Input ~ 0
 aPHIb
-Text HLabel 1050 6100 0    50   Input ~ 0
+Text HLabel 1050 4000 0    50   Input ~ 0
 aPHI
 Text HLabel 1050 7100 0    50   Input ~ 0
@@
 Text Label 2350 3900 0    50   ~ 0
 aLOAD33
-Text Label 2350 4000 0    50   ~ 0
+Text Label 2350 3800 0    50   ~ 0
 aSCANIN33
 Text Label 2350 4100 0    50   ~ 0
@@
 Text Label 1750 1450 0    50   ~ 0
 aSCSEL33
-Text Label 2350 6100 0    50   ~ 0
+Text Label 2350 4000 0    50   ~ 0
 aPHI33
 Text Label 1750 1350 0    50   ~ 0
 aPHI33
-Text Label 2350 6200 0    50   ~ 0
+Text Label 2350 5000 0    50   ~ 0
 aPHIb33
-Text Label 2350 4900 0    50   ~ 0
+Text Label 2350 5100 0    50   ~ 0
 Clock33
 Text Label 2350 6300 0    50   ~ 0
@@
 	0    -1   -1   0
 $EndComp
-Text Label 2350 5200 0    50   ~ 0
+Text Label 2350 6200 0    50   ~ 0
 3WB_CLK33
-Text Label 2350 5100 0    50   ~ 0
+Text Label 2350 6100 0    50   ~ 0
 3WB_ENB33
-Text Label 2350 5000 0    50   ~ 0
+Text Label 2350 6000 0    50   ~ 0
 3WB_DATA33
 Text Label 1750 2350 0    50   ~ 0
@@
 Text Label 1750 2150 0    50   ~ 0
 3WB_DATA33
-Text Label 2350 6000 0    50   ~ 0
+Text Label 2350 5200 0    50   ~ 0
 GPO_ZERO33
 $Comp
@@
 NoConn ~ 1050 7400
 NoConn ~ 1050 7300
-NoConn ~ 1050 3800
-NoConn ~ 2350 3800
+NoConn ~ 1050 4900
+NoConn ~ 2350 4900
 NoConn ~ 2350 7200
 NoConn ~ 1050 7200
