File: scum3c_devboard_large/scum3c-devboard.kicad_pcb (KiCad board)
At the start: 2 copper layers, 46.1 x 73.1 mm, 63 parts, among them J1 CONSMA001-G, J10 Conn_02x01, J11 Conn_01x01, J12 Conn_02x01, J13 Conn_02x01, J14 Conn_01x01_Male, J15 Conn_01x01_Male, J16 Conn_02x01, J17 Conn_02x01, J2 47346-0001, J3 Conn_02x06_Odd_Even, J4 Conn_01x22, J5 Conn_02x05_Odd_Even, J6 Conn_01x03, J7 Conn_01x03, J8 Conn_01x03, J9 Conn_02x03_Odd_Even, U1 Perfboard, U10 74AVCH4T245D,118, U11 74AVCH4T245D,118, U12 S-85S1AB18-I6T1U, U13 74AVCH4T245D,118, U2 FT231XS-U, U3 74AVC1T45GS-Q100H, U4 74AVC1T45GS-Q100H, U5 ICM-20948, U6 S-85S1AB10-I6T1U, U7 S-85S1AB15-I6T1U, U8 scum3, U9 74AVCH4T245D,118

Commit message: ready for review
Parts:
- removed J10, J12, J13, J16, J17: Conn_02x01, Connector_PinHeader_2.54mm:PinHeader_2x01_P2.54mm_Vertical
- removed J11: Conn_01x01, Connector_PinHeader_2.54mm:PinHeader_1x01_P2.54mm_Vertical
- removed J14, J15: Conn_01x01_Male, Connector_PinHeader_2.54mm:PinHeader_1x01_P2.54mm_Vertical
- removed J7, J8: Conn_01x03, Connector_PinHeader_2.54mm:PinHeader_1x03_P2.54mm_Vertical
- added C13: C, Capacitor_SMD:C_0402_1005Metric, F.Cu at (196.7, 90.4)
- added U14: 74AVCH4T245D,118, downloaded_libs:SOIC127P600X175-16N, F.Cu at (215.6, 74.3)
- added U15: 74AVCH4T245D,118, downloaded_libs:SOIC127P600X175-16N, F.Cu at (199.7, 73.8)
- J2: value 47346-0001 -> Conn_02x04_Odd_Even; footprint Connector_USB:USB_Micro-B_Molex_47346-0001 -> Connector_PinHeader_2.54mm:PinHeader_2x04_P2.54mm_Vertical
- J3: value Conn_02x06_Odd_Even -> Conn_02x10_Odd_Even; footprint Connector_PinHeader_2.54mm:PinHeader_2x06_P2.54mm_Vertical -> Connector_PinHeader_2.54mm:PinHeader_2x10_P2.54mm_Vertical
- J4: value Conn_01x22 -> Conn_02x13_Odd_Even; footprint SCUM:Teensy_Connector -> Connector_PinHeader_2.54mm:PinHeader_2x13_P2.54mm_Vertical
- J5: value Conn_02x05_Odd_Even -> 1050170001; footprint Connector_PinHeader_2.54mm:PinHeader_2x05_P2.54mm_Vertical -> SCUM:MOLEX_1050170001
- J6: value Conn_01x03 -> Conn_01x24; footprint Connector_PinHeader_2.54mm:PinHeader_1x03_P2.54mm_Vertical -> Connector_PinSocket_2.54mm:PinSocket_1x24_P2.54mm_Vertical
- moved U9 49.3 mm to (225.4, 74.3)
- moved J4 46.6 mm to (191.9, 97.4)
- moved J6 46.5 mm to (232.8, 132.3), turned to 180 degrees
- moved U11 38.0 mm to (224.0, 123.6)
- moved J5 30.9 mm to (192.3, 86.6), turned to 270 degrees
- moved C6 20.6 mm to (198.9, 81.1), turned to 180 degrees
- moved C5 17.5 mm to (198.8, 82.3), turned to 180 degrees
- moved R1 16.3 mm to (198.8, 83.5), turned to 180 degrees
- moved R4 15.1 mm to (208.0, 80.7), turned to 270 degrees
- moved J2 14.5 mm to (191.5, 68.7), turned to 0 degrees
- moved D1 14.2 mm to (199.3, 85.1), turned to 270 degrees
- moved U2 12.0 mm to (203.6, 83.7), turned to 0 degrees
- moved D2 12.0 mm to (208.0, 83.0), turned to 270 degrees
- moved U10 10.8 mm to (225.4, 85.5)
- moved C26 10.3 mm to (207.6, 75.9)
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Connections:
- C26 pad 1: +VIN -> +VIN_IMU
- C27 pad 1: +V18IO -> +V18IO_IMU
- C28 pad 1: +VBAT' -> +15VIN
- C5 pad 1: +UART33 -> +USB33
- C6 pad 1: +UART33 -> +USB33
- J2 pad 1: Net-(C2-Pad1) -> GND
- J2 pad 2: /UART/D_N -> GND
- J2 pad 3: /UART/D_P -> /ADC_IN
- J2 pad 4: Net-(J2-Pad4) -> /ADC_LDO_OUT
- J2 pad 5: GND -> +VIN
- J2 pad 6: (no net) -> +VIN_IMU
- J3 pad 1: /GPIO4 -> /GPIO8
- J3 pad 10: /GPIO13 -> /GPIO5
- J3 pad 11: /GPIO14 -> /GPIO6
- J3 pad 12: /GPIO15 -> /GPIO7
- J3 pad 2: /GPIO5 -> /GPIO1
- J3 pad 3: /GPIO6 -> /GPIO9
- J3 pad 4: /GPIO7 -> /GPIO1
- J3 pad 5: /GPIO8 -> /GPIO0
- J3 pad 6: /GPIO9 -> /GPIO1
- J3 pad 7: /GPIO10 -> /GPIO2
- J3 pad 8: /GPIO11 -> /GPIO3
- J3 pad 9: /GPIO12 -> /GPIO4
- J5 pad 1: /Boot_Source_Sel -> Net-(C2-Pad1)
- J5 pad 2: +VDDD -> /UART/D_N
- J5 pad 3: +VDDD' -> /UART/D_P
- J5 pad 4: GND -> Net-(J5-Pad4)
- J5 pad 5: +VDDIO' -> GND
- J6 pad 1: +VIN -> Net-(J6-Pad1)
- J6 pad 2: +VDDIO' -> Net-(J6-Pad2)
- J6 pad 3: +VBAT' -> +TEENSY33
- L3 pad 1: +VBAT' -> +15VIN
- R1 pad 1: +UART33 -> +USB33
- R1 pad 2: Net-(D1-Pad1) -> Net-(D1-Pad2)
- R4 pad 1: +UART33 -> +USB33
- R4 pad 2: Net-(D2-Pad1) -> Net-(D2-Pad2)
- U10 pad 10: /Teensy Connections/3WB_CLK33 -> /Teensy Connections/GPO_ZERO33
- U10 pad 11: /Teensy Connections/3WB_ENB33 -> /Teensy Connections/Clock33
- U10 pad 12: /Teensy Connections/3WB_DATA33 -> /Teensy Connections/aPHIb33
- U10 pad 13: /Teensy Connections/Clock33 -> Net-(U10-Pad13)
- U10 pad 4: /Clock -> Net-(U10-Pad4)
- U10 pad 5: /3WB_DATA -> /aPHIb
- U10 pad 6: /3WB_ENB -> /Clock
- U10 pad 7: /3WB_CLK -> /GPO_ZERO
- U11 pad 11: /Teensy Connections/aPHIb33 -> /Teensy Connections/3WB_CLK33
- U11 pad 12: /Teensy Connections/aPHI33 -> /Teensy Connections/3WB_ENB33
- U11 pad 13: /Teensy Connections/sReset33 -> /Teensy Connections/3WB_DATA33
- U11 pad 4: /sReset -> /3WB_DATA
- U11 pad 5: /aPHI -> /3WB_ENB
- U11 pad 6: /aPHIb -> /3WB_CLK
- U2 pad 10: Net-(D1-Pad2) -> Net-(D1-Pad1)
- U2 pad 13: +UART33 -> +USB33
- U2 pad 14: +UART33 -> +USB33
- U2 pad 17: Net-(D2-Pad2) -> Net-(D2-Pad1)
- U2 pad 3: +UART33 -> +USB33
- U5 pad 13: +VIN -> +VIN_IMU
- U5 pad 22: /GPIO15 -> /GPIO15_IMU
- U5 pad 23: /GPIO14 -> /GPIO14_IMU
- U5 pad 24: /GPIO12 -> /GPIO12_IMU
- U5 pad 8: +V18IO -> +V18IO_IMU
- U5 pad 9: /GPIO13 -> /GPIO13_IMU
- U7 pad 1: +VBAT' -> +15VIN
- U8 pad 17: +VBAT -> +VBATSCuM
- U8 pad 26: +VBAT -> +VBATSCuM
- U8 pad 36: +VDDIO -> +VDDIOSCuM
- U8 pad 4: +VBAT -> +VBATSCuM
- U8 pad 53: Net-(J15-Pad1) -> /ADC_LDO_OUT
- U8 pad 54: Net-(J14-Pad1) -> /ADC_IN
- U8 pad 57: Net-(U8-Pad57) -> /GPO_ZERO
- U8 pad 59: +VBAT -> +VBATSCuM
- U8 pad 62: +VBAT -> +VBATSCuM
- U8 pad 80: /sReset -> Net-(U8-Pad80)
- U9 pad 11: /Teensy Connections/aSCANIN33 -> /Teensy Connections/aPHI33
- U9 pad 13: Net-(U9-Pad13) -> /Teensy Connections/aSCANIN33
- U9 pad 4: Net-(U9-Pad4) -> /aSCANIN
- U9 pad 6: /aSCANIN -> /aPHI
Routing:
- net +VDDIOSCuM: track 0.00 -> 68.5 mm, vias 0 -> 1
- net /Tx33: track 11.2 -> 72.3 mm
- net /ADC_LDO_OUT: track 0.00 -> 60.1 mm, vias 0 -> 1
- net /Rx33: track 9.49 -> 65.3 mm
- net +VBAT': track 55.5 -> 0.00 mm
- net +VBATSCuM: track 0.00 -> 55.2 mm, vias 0 -> 2
- net /ADC_IN: track 0.00 -> 54.4 mm, vias 0 -> 1
- net +VDDIO: track 53.5 -> 101.8 mm, vias 2 -> 3
- net +UART33: track 43.3 -> 0.00 mm, vias 1 -> 0
- net +USB33: track 0.00 -> 41.7 mm, vias 0 -> 1
- net +15VIN: track 0.00 -> 35.3 mm, vias 0 -> 1
- net /Teensy Connections/sReset33: track 35.0 -> 0.00 mm
- net /Teensy Connections/aLOAD33: track 48.4 -> 14.1 mm, vias 1 -> 0
- net /sReset: track 31.8 -> 0.00 mm, vias 2 -> 0
- net /hReset: track 15.5 -> 46.7 mm, vias 1 -> 2
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- added copper zone on F.Cu, net Net-(C13-Pad1)
Other:
- board size 46.1 x 73.1 mm -> 46.1 x 83.1 mm
- board text added: "ADC"
- board text added: "Current Measure"
- board text added: "GPIO0"
- board text added: "GPIO15"
- board text added: "IMU Current"
- board text added: "Lighthouse"
- board text added: "Teensy 6V In"
- board text added: "VDDIO Sel"
- board text added: "VIN"
- board text added: "VIN Sel"
- board text removed: "GPIO"
- board text removed: "IBAT"
- board text removed: "IDDD"
- board text removed: "IDDIO"
- board text removed: "TEENSY"
- board text removed: "Teensy Pin A9"
- board text removed: "UART"
- board text removed: "VDDD Select"
- board text removed: "VDDIO Select"
- board text removed: "VIN Select"
