File: scum3c_devboard_large/scum3c-devboard.sch (KiCad schematic (older format))
At the start: 34 parts, among them J1 CONSMA001-SMD-G-T, J10 Conn_01x02, J11 Conn_01x01, J3 Conn_02x06_Odd_Even, J5 Conn_02x04_Odd_Even, J6 Conn_01x03, J7 Conn_01x03, J8 Conn_01x03, U1 Perfboard, U12 S-85S1AB18-I6T1U, U5 ICM-20948, U6 S-85S1AB10-I6T1U, U7 S-85S1AB15-I6T1U

Commit message: With through-hole antenna
Parts:
- removed J1: CONSMA001-SMD-G-T, downloaded_libs:LINX_CONSMA001-SMD-G-T, symbol CONSMA001-SMD-G-T:CONSMA001-SMD-G-T
- added J1: CONSMA001-G, downloaded_libs:LINX_CONSMA001-G, symbol CONSMA001-G:CONSMA001-G
- E1: renamed from E?; footprint ANT_2450AT45A100E -> downloaded_libs:ANT_2450AT45A100E
Changed lines of the file:
@@
 Text Notes 3100 7750 0    50   ~ 0
 Antenna
-$Comp
-L CONSMA001-SMD-G-T:CONSMA001-SMD-G-T J1
-U 1 1 5FA2C43F
-P 2300 7050
-F 0 "J1" H 2293 7257 50  0000 C CNN
-F 1 "CONSMA001-SMD-G-T" H 2293 7166 50  0000 C CNN
-F 2 "downloaded_libs:LINX_CONSMA001-SMD-G-T" H 2300 7050 50  0001 L BNN
-F 3 "10.4 mm" H 2300 7050 50  0001 L BNN
-F 4 "F" H 2300 7050 50  0001 L BNN "Field4"
-F 5 "Manufacturer Recommendations" H 2300 7050 50  0001 L BNN "Field5"
-F 6 "Linx" H 2300 7050 50  0001 L BNN "Field6"
-	1    2300 7050
-	1    0    0    -1
-$EndComp
 Wire Wire Line
 	2400 7050 2400 7100
@@
 Wire Wire Line
 	2550 7100 2550 7450
-Connection ~ 2400 7050
 Wire Wire Line
 	2400 7050 2700 7050
@@
 Text Label 6500 2350 0    50   ~ 0
 PVSS1.5
-NoConn ~ 3100 7350
 Wire Notes Line
 	6050 550  9700 550
@@
 Connection ~ 3100 1700
 $Comp
-L 2450AT45A100E:2450AT45A100E E?
+L 2450AT45A100E:2450AT45A100E E1
 U 1 1 6011A2BA
 P 3250 7200
-F 0 "E?" H 3000 7300 50  0000 L CNN
+F 0 "E1" H 3000 7300 50  0000 L CNN
 F 1 "2450AT45A100E" H 2650 7200 50  0000 L CNN
-F 2 "ANT_2450AT45A100E" H 3250 7200 50  0001 L BNN
+F 2 "downloaded_libs:ANT_2450AT45A100E" H 3250 7200 50  0001 L BNN
 F 3 "" H 3250 7200 50  0001 L BNN
 F 4 "Johanson" H 3250 7200 50  0001 L BNN "MANUFACTURER"
@@
 	3250 7450 2850 7450
 Connection ~ 2850 7450
+$Comp
+L CONSMA001-G:CONSMA001-G J1
+U 1 1 6047CDDD
+P 2300 7050
+F 0 "J1" H 2293 7257 50  0000 C CNN
+F 1 "CONSMA001-G" H 2293 7166 50  0000 C CNN
+F 2 "downloaded_libs:LINX_CONSMA001-G" H 2300 7050 50  0001 L BNN
+F 3 "" H 2300 7050 50  0001 L BNN
+F 4 "Linx Technologies" H 2300 7050 50  0001 L BNN "MANUFACTURER"
+F 5 "D" H 2300 7050 50  0001 L BNN "PARTREV"
+F 6 "Manufacturer Recommendations" H 2300 7050 50  0001 L BNN "STANDARD"
+F 7 "9.79mm" H 2300 7050 50  0001 L BNN "MAXIMUM_PACKAGE_HEIGHT"
+	1    2300 7050
+	1    0    0    -1
+$EndComp
+Connection ~ 2400 7050
+NoConn ~ 2850 2600
 $EndSCHEMATC

Commit message: ensuring large board up to date with master
Changed lines of the file:
@@
 F2 "RsRx" I L 800 7200 50
 F3 "RsTx" O R 1400 7200 50
-F4 "VBAT_USB" I R 1400 7550 50
 F5 "RsTxTeensy" I R 1400 7400 50
 F6 "RsRxTeensy" I L 800 7300 50
@@
 	1    0    0    -1
 $EndComp
-Text Label 1400 7550 0    50   ~ 0
-VBAT_USB
 $Comp
 L Connector_Generic:Conn_01x03 J8

Commit message: Suggested changes
Parts:
- removed J10: Conn_01x02, Connector_PinHeader_2.54mm:PinHeader_1x02_P2.54mm_Vertical, symbol Connector_Generic:Conn_01x02
- removed J5: Conn_02x04_Odd_Even, Connector_PinHeader_2.54mm:PinHeader_2x04_P2.54mm_Vertical, symbol Connector_Generic:Conn_02x04_Odd_Even
- removed R5, R6: 10k, Resistor_SMD:R_0402_1005Metric, symbol Device:R
- added J10, J12, J13, J16, J17: Conn_02x01, Connector_PinHeader_2.54mm:PinHeader_2x01_P2.54mm_Vertical, symbol Connector_Generic:Conn_02x01
- added J5: Conn_02x05_Odd_Even, Connector_PinHeader_2.54mm:PinHeader_2x05_P2.54mm_Vertical, symbol Connector_Generic:Conn_02x05_Odd_Even
- J1: symbol CONSMA001-G:CONSMA001-G -> SCUM:CONSMA001-G-CONSMA001-G
- U1: symbol scum3c-devboard-rescue:Perfboard-SCUM -> SCUM:Perfboard
Connections:
- net +VBAT: now also J10.2 (Pin_2); no longer C28.1, J6.3 (Pin_3), J7.3 (Pin_3), L3.1, U7.1 (VOUT)
- net +VDDD: now also J13.2 (Pin_2), J5.2 (Pin_2); no longer J7.2 (Pin_2)
- net +VDDIO: now also J12.2 (Pin_2); no longer J6.2 (Pin_2)
- net +VIN: now also J5.9 (Pin_9)
- net Boot_Source_Sel: now also J5.1 (Pin_1)
- net GND: now also J5.10 (Pin_10), J5.4 (Pin_4), J5.6 (Pin_6), J5.8 (Pin_8)
- net GPIO1: now also J16.1 (Pin_1), J17.1 (Pin_1)
- net GPIO12: now also U5.24 (SDA/SDI); no longer U5.9 (AD0/SDO)
- net GPIO13: now also U5.9 (AD0/SDO); no longer U5.24 (SDA/SDI)
- net GPIO8: now also J16.2 (Pin_2)
- net GPIO9: now also J17.2 (Pin_2)
- net 1Vin renamed +1VIN
- new net: U1.11, U1.21, U1.31, U1.41
- new net: U1.12, U1.22, U1.32, U1.42
- new net: U1.13, U1.23, U1.33, U1.43
- new net: U1.14, U1.24, U1.34, U1.44
- new net: U1.15, U1.25, U1.35, U1.45
- new net: U1.16, U1.26, U1.36, U1.46
- new net: U1.17, U1.27, U1.37, U1.47
- new net: U1.18, U1.28, U1.38, U1.48
- new net +VBAT': C28.1, J10.1 (Pin_1), J5.7 (Pin_7), J6.3 (Pin_3), J7.3 (Pin_3), L3.1, U7.1 (VOUT)
- new net +VDDD': J13.1 (Pin_1), J5.3 (Pin_3), J7.2 (Pin_2)
- new net +VDDIO': J12.1 (Pin_1), J5.5 (Pin_5), J6.2 (Pin_2)
- no-connect marks 5 -> 15
Other:
- note added: "Current Measurement"
- moved on the sheet: J7, J8

Commit message: switching computers
Parts:
- removed J10, J12, J13, J16, J17: Conn_02x01, Connector_PinHeader_2.54mm:PinHeader_2x01_P2.54mm_Vertical, symbol Connector_Generic:Conn_02x01
- removed J11: Conn_01x01, Connector_PinHeader_2.54mm:PinHeader_1x01_P2.54mm_Vertical, symbol Connector_Generic:Conn_01x01
- removed J3: Conn_02x06_Odd_Even, Connector_PinHeader_2.54mm:PinHeader_2x06_P2.54mm_Vertical, symbol Connector_Generic:Conn_02x06_Odd_Even
- removed J5: Conn_02x05_Odd_Even, Connector_PinHeader_2.54mm:PinHeader_2x05_P2.54mm_Vertical, symbol Connector_Generic:Conn_02x05_Odd_Even
- removed J6, J7, J8: Conn_01x03, Connector_PinHeader_2.54mm:PinHeader_1x03_P2.54mm_Vertical, symbol Connector_Generic:Conn_01x03
- added J2: Conn_02x04_Odd_Even, Connector_PinHeader_2.54mm:PinHeader_2x04_P2.54mm_Vertical, symbol Connector_Generic:Conn_02x04_Odd_Even
- added J3: Conn_02x10_Odd_Even, Connector_PinHeader_2.54mm:PinHeader_2x10_P2.54mm_Vertical, symbol Connector_Generic:Conn_02x10_Odd_Even
- added J4: Conn_02x13_Odd_Even, Connector_PinHeader_2.54mm:PinHeader_2x13_P2.54mm_Vertical, symbol Connector_Generic:Conn_02x13_Odd_Even
- added U14, U15: 74AVCH4T245D,118, downloaded_libs:SOIC127P600X175-16N, symbol SCUM:74AVCH4T245D,118
Connections:
- net +1VIN: now also J4.15 (Pin_15)
- net +TEENSY33: now also J4.6 (Pin_6)
- net +V18IO: now also J2.7 (Pin_7), J4.8 (Pin_8), U14.1 (VCC(A)), U15.1 (VCC(A)), U15.2 (1DIR); no longer C27.1, U5.8 (VDDIO)
- net +VBAT: now also J4.12 (Pin_12), J4.14 (Pin_14), J4.23 (Pin_23), J4.3 (Pin_3)
- net +VDDD: now also J4.16 (Pin_16), J4.18 (Pin_18), J4.19 (Pin_19)
- net +VDDIO: now also J4.1 (Pin_1), J4.10 (Pin_10), J4.21 (Pin_21), U14.16 (VCC(B)), U15.16 (VCC(B))
- net +VIN: now also J2.5 (Pin_5), J4.25 (Pin_25), J4.5 (Pin_5), J4.9 (Pin_9); no longer C26.1, U5.13 (VDD)
- net Boot_Source_Sel: now also J4.17 (Pin_17)
- net GND: now also J2.1 (Pin_1), J2.2 (Pin_2), J4.11 (Pin_11), J4.20 (Pin_20), J4.22 (Pin_22), J4.24 (Pin_24), J4.26 (Pin_26), U14.14 (2OE'), U14.15 (1OE'), U14.2 (1DIR), U14.3 (2DIR), U14.8 (GND-1), U14.9 (GND), U15.14 (2OE'), U15.15 (1OE'), U15.3 (2DIR), U15.8 (GND-1), U15.9 (GND)
- net GPIO0: now also J3.5 (Pin_5)
- net GPIO1: now also J3.2 (Pin_2), J3.4 (Pin_4), J3.6 (Pin_6)
- net GPIO10: now also J3.15 (Pin_15)
- net GPIO11: now also J3.16 (Pin_16)
- net GPIO12: now also J3.17 (Pin_17), U14.11 (2B1); no longer U5.24 (SDA/SDI)
- net GPIO13: now also J3.18 (Pin_18), U15.12 (1B2); no longer U5.9 (AD0/SDO)
- net GPIO14: now also J3.19 (Pin_19), U14.12 (1B2); no longer U5.23 (SCL/SCLK)
- net GPIO15: now also J3.20 (Pin_20), U14.10 (2B2); no longer U5.22 (~CS)
- net GPIO2: now also J3.7 (Pin_7)
- net GPIO3: now also J3.8 (Pin_8)
- net GPIO4: now also J3.9 (Pin_9)
- net GPIO5: now also J3.10 (Pin_10)
- net GPIO6: now also J3.11 (Pin_11)
- net GPIO7: now also J3.12 (Pin_12)
- net GPIO8: now also J3.1 (Pin_1), J3.13 (Pin_13)
- net GPIO9: now also J3.14 (Pin_14), J3.3 (Pin_3)
- net +VBAT' renamed +15VIN
- net +15VIN: now also J4.13 (Pin_13)
- new net +USB33: J4.7 (Pin_7)
- new net +V18IO_IMU: C27.1, J2.8 (Pin_8), U5.8 (VDDIO)
- new net +VBATSCuM: J4.4 (Pin_4)
- new net +VDDIOSCuM: J4.2 (Pin_2)
- new net +VIN_IMU: C26.1, J2.6 (Pin_6), U5.13 (VDD)
- new net ADC_IN: J2.3 (Pin_3)
- new net ADC_LDO_OUT: J2.4 (Pin_4)
- new net GPIO12_IMU: U14.6 (2A1), U5.24 (SDA/SDI)
- new net GPIO13_IMU: U15.5 (1A2), U5.9 (AD0/SDO)
- new net GPIO14_IMU: U14.5 (1A2), U5.23 (SCL/SCLK)
- new net GPIO15_IMU: U14.7 (2A2), U5.22 (~CS)
- no-connect marks 15 -> 23
Other:
- note added: "ADC/IMU Pins"
- note added: "GPIO"
- note added: "IMU Level Shifters"
- note added: "Voltage Pins"
- note removed: "Connectors"
- note removed: "Current Measurement"
- moved on the sheet: H1, H2, H3, H4

Commit message: ready for review
Connections:
- net +15VIN: now also J4.9 (Pin_9); no longer J4.13 (Pin_13)
- net +TEENSY33: now also J4.2 (Pin_2); no longer J4.6 (Pin_6)
- net +USB33: now also J4.3 (Pin_3); no longer J4.7 (Pin_7)
- net +V18IO: now also J4.4 (Pin_4); no longer J4.8 (Pin_8)
- net +VBAT: now also J4.10 (Pin_10), J4.11 (Pin_11), J4.8 (Pin_8); no longer J4.12 (Pin_12), J4.14 (Pin_14), J4.3 (Pin_3)
- net +VBATSCuM: now also J4.12 (Pin_12); no longer J4.4 (Pin_4)
- net +VDDIO: now also J4.13 (Pin_13), J4.6 (Pin_6); no longer J4.1 (Pin_1), J4.10 (Pin_10)
- net +VDDIOSCuM: now also J4.14 (Pin_14); no longer J4.2 (Pin_2)
- net +VIN: now also J4.1 (Pin_1); no longer J4.9 (Pin_9)
- net GND: now also J4.7 (Pin_7); no longer J4.11 (Pin_11)
Changed lines of the file:
@@
 EESchema Schematic File Version 4
 LIBS:scum3c-devboard-cache
-EELAYER 30 0
+EELAYER 26 0
 EELAYER END
 $Descr A 11000 8500
@@
 L SCUM:+VBAT #PWR0107
 U 1 1 608EB617
-P 2800 5550
-F 0 "#PWR0107" H 2800 5400 50  0001 C CNN
-F 1 "+VBAT" V 2815 5678 50  0000 L CNN
-F 2 "" H 2800 5550 50  0001 C CNN
-F 3 "" H 2800 5550 50  0001 C CNN
-	1    2800 5550
+P 2800 5350
+F 0 "#PWR0107" H 2800 5200 50  0001 C CNN
+F 1 "+VBAT" V 2815 5478 50  0000 L CNN
+F 2 "" H 2800 5350 50  0001 C CNN
+F 3 "" H 2800 5350 50  0001 C CNN
+	1    2800 5350
 	0    1    1    0
 $EndComp
@@
 L SCUM:+VBAT #PWR0110
 U 1 1 608EBC39
-P 2800 5450
-F 0 "#PWR0110" H 2800 5300 50  0001 C CNN
-F 1 "+VBAT" V 2815 5578 50  0000 L CNN
-F 2 "" H 2800 5450 50  0001 C CNN
-F 3 "" H 2800 5450 50  0001 C CNN
-	1    2800 5450
+P 2800 5250
+F 0 "#PWR0110" H 2800 5100 50  0001 C CNN
+F 1 "+VBAT" V 2815 5378 50  0000 L CNN
+F 2 "" H 2800 5250 50  0001 C CNN
+F 3 "" H 2800 5250 50  0001 C CNN
+	1    2800 5250
 	0    1    1    0
 $EndComp
@@
 L SCUM:+15VIN #PWR0120
 U 1 1 608EEC94
-P 2300 5550
-F 0 "#PWR0120" H 2300 5400 50  0001 C CNN
-F 1 "+15VIN" V 2315 5678 50  0000 L CNN
-F 2 "" H 2300 5550 50  0001 C CNN
-F 3 "" H 2300 5550 50  0001 C CNN
-	1    2300 5550
-	0    -1   -1   0
-$EndComp
-$Comp
-L power:GND #PWR0122
-U 1 1 608F078D
-P 2300 5450
-F 0 "#PWR0122" H 2300 5200 50  0001 C CNN
-F 1 "GND" V 2305 5322 50  0000 R CNN
-F 2 "" H 2300 5450 50  0001 C CNN
-F 3 "" H 2300 5450 50  0001 C CNN
-	1    2300 5450
-	0    1    1    0
-$EndComp
-$Comp
-L SCUM:+VIN #PWR0124
-U 1 1 608F0F40
 P 2300 5350
-F 0 "#PWR0124" H 2300 5200 50  0001 C CNN
-F 1 "+VIN" V 2315 5477 50  0000 L CNN
+F 0 "#PWR0120" H 2300 5200 50  0001 C CNN
+F 1 "+15VIN" V 2315 5478 50  0000 L CNN
 F 2 "" H 2300 5350 50  0001 C CNN
 F 3 "" H 2300 5350 50  0001 C CNN
@@
 $EndComp
 $Comp
-L SCUM:+VDDIO #PWR0132
-U 1 1 608F126B
-P 2800 5350
-F 0 "#PWR0132" H 2800 5200 50  0001 C CNN
-F 1 "+VDDIO" V 2815 5478 50  0000 L CNN
-F 2 "" H 2800 5350 50  0001 C CNN
-F 3 "" H 2800 5350 50  0001 C CNN
-	1    2800 5350
-	0    1    1    0
-$EndComp
-$Comp
-L SCUM:+V18IO #PWR0150
-U 1 1 608F2648
-P 2800 5250
-F 0 "#PWR0150" H 2800 5100 50  0001 C CNN
-F 1 "+V18IO" V 2815 5378 50  0000 L CNN
-F 2 "" H 2800 5250 50  0001 C CNN
-F 3 "" H 2800 5250 50  0001 C CNN
-	1    2800 5250
-	0    1    1    0
-$EndComp
-$Comp
-L SCUM:+USB33 #PWR0151
-U 1 1 608F483E
+L power:GND #PWR0122
+U 1 1 608F078D
 P 2300 5250
-F 0 "#PWR0151" H 2300 5100 50  0001 C CNN
-F 1 "+USB33" V 2315 5377 50  0000 L CNN
+F 0 "#PWR0122" H 2300 5000 50  0001 C CNN
+F 1 "GND" V 2305 5122 50  0000 R CNN
 F 2 "" H 2300 5250 50  0001 C CNN
 F 3 "" H 2300 5250 50  0001 C CNN
 	1    2300 5250
-	0    -1   -1   0
-$EndComp
-$Comp
-L SCUM:+VIN #PWR0152
-U 1 1 608F5209
+	0    1    1    0
+$EndComp
+$Comp
+L SCUM:+VIN #PWR0124
+U 1 1 608F0F40
 P 2300 5150
-F 0 "#PWR0152" H 2300 5000 50  0001 C CNN
+F 0 "#PWR0124" H 2300 5000 50  0001 C CNN
 F 1 "+VIN" V 2315 5277 50  0000 L CNN
 F 2 "" H 2300 5150 50  0001 C CNN
@@
 $EndComp
 $Comp
-L SCUM:+TEENSY33 #PWR0154
-U 1 1 608F5F6B
+L SCUM:+VDDIO #PWR0132
+U 1 1 608F126B
 P 2800 5150
-F 0 "#PWR0154" H 2800 5000 50  0001 C CNN
-F 1 "+TEENSY33" V 2815 5278 50  0000 L CNN
+F 0 "#PWR0132" H 2800 5000 50  0001 C CNN
+F 1 "+VDDIO" V 2815 5278 50  0000 L CNN
 F 2 "" H 2800 5150 50  0001 C CNN
 F 3 "" H 2800 5150 50  0001 C CNN
@@
 $EndComp
 $Comp
-L SCUM:+VDDIOSCuM #PWR0170
-U 1 1 608F684F
+L SCUM:+V18IO #PWR0150
+U 1 1 608F2648
+P 2800 5050
+F 0 "#PWR0150" H 2800 4900 50  0001 C CNN
+F 1 "+V18IO" V 2815 5178 50  0000 L CNN
+F 2 "" H 2800 5050 50  0001 C CNN
+F 3 "" H 2800 5050 50  0001 C CNN
+	1    2800 5050
+	0    1    1    0
+$EndComp
+$Comp
+L SCUM:+USB33 #PWR0151
+U 1 1 608F483E
+P 2300 5050
+F 0 "#PWR0151" H 2300 4900 50  0001 C CNN
+F 1 "+USB33" V 2315 5177 50  0000 L CNN
+F 2 "" H 2300 5050 50  0001 C CNN
+F 3 "" H 2300 5050 50  0001 C CNN
+	1    2300 5050
+	0    -1   -1   0
+$EndComp
+$Comp
+L SCUM:+VIN #PWR0152
+U 1 1 608F5209
+P 2300 4950
+F 0 "#PWR0152" H 2300 4800 50  0001 C CNN
+F 1 "+VIN" V 2315 5077 50  0000 L CNN
+F 2 "" H 2300 4950 50  0001 C CNN
+F 3 "" H 2300 4950 50  0001 C CNN
+	1    2300 4950
+	0    -1   -1   0
+$EndComp
+$Comp
+L SCUM:+TEENSY33 #PWR0154
+U 1 1 608F5F6B
 P 2800 4950
-F 0 "#PWR0170" H 2800 4800 50  0001 C CNN
-F 1 "+VDDIOSCuM" V 2815 5078 50  0000 L CNN
+F 0 "#PWR0154" H 2800 4800 50  0001 C CNN
+F 1 "+TEENSY33" V 2815 5078 50  0000 L CNN
 F 2 "" H 2800 4950 50  0001 C CNN
 F 3 "" H 2800 4950 50  0001 C CNN
@@
 $EndComp
 $Comp
+L SCUM:+VDDIOSCuM #PWR0170
+U 1 1 608F684F
+P 2800 5550
+F 0 "#PWR0170" H 2800 5400 50  0001 C CNN
+F 1 "+VDDIOSCuM" V 2815 5678 50  0000 L CNN
+F 2 "" H 2800 5550 50  0001 C CNN
+F 3 "" H 2800 5550 50  0001 C CNN
+	1    2800 5550
+	0    1    1    0
+$EndComp
+$Comp
 L SCUM:+VBATSCuM #PWR0176
 U 1 1 608F8177
-P 2800 5050
-F 0 "#PWR0176" H 2800 4900 50  0001 C CNN
-F 1 "+VBATSCuM" V 2815 5178 50  0000 L CNN
-F 2 "" H 2800 5050 50  0001 C CNN
-F 3 "" H 2800 5050 50  0001 C CNN
-	1    2800 5050
+P 2800 5450
+F 0 "#PWR0176" H 2800 5300 50  0001 C CNN
+F 1 "+VBATSCuM" V 2815 5578 50  0000 L CNN
+F 2 "" H 2800 5450 50  0001 C CNN
+F 3 "" H 2800 5450 50  0001 C CNN
+	1    2800 5450
 	0    1    1    0
 $EndComp
@@
 L SCUM:+VBAT #PWR0190
 U 1 1 608F910B
-P 2300 5050
-F 0 "#PWR0190" H 2300 4900 50  0001 C CNN
-F 1 "+VBAT" V 2315 5178 50  0000 L CNN
-F 2 "" H 2300 5050 50  0001 C CNN
-F 3 "" H 2300 5050 50  0001 C CNN
-	1    2300 5050
+P 2300 5450
+F 0 "#PWR0190" H 2300 5300 50  0001 C CNN
+F 1 "+VBAT" V 2315 5578 50  0000 L CNN
+F 2 "" H 2300 5450 50  0001 C CNN
+F 3 "" H 2300 5450 50  0001 C CNN
+	1    2300 5450
 	0    -1   -1   0
 $EndComp
@@
 L SCUM:+VDDIO #PWR0193
 U 1 1 608F9BD6
-P 2300 4950
-F 0 "#PWR0193" H 2300 4800 50  0001 C CNN
-F 1 "+VDDIO" V 2315 5077 50  0000 L CNN
-F 2 "" H 2300 4950 50  0001 C CNN
-F 3 "" H 2300 4950 50  0001 C CNN
-	1    2300 4950
-	0    -1   -1   0
-$EndComp
+P 2300 5550
+F 0 "#PWR0193" H 2300 5400 50  0001 C CNN
+F 1 "+VDDIO" V 2315 5677 50  0000 L CNN
+F 2 "" H 2300 5550 50  0001 C CNN
+F 3 "" H 2300 5550 50  0001 C CNN
+	1    2300 5550
+	0    -1   -1   0
+$EndComp
