File: mccoy/scumsheet.sch (KiCad schematic (older format))
At the start: 19 parts, among them J10 through_hole, J11 through_hole, J12 through_hole, J13 through_hole, J14 through_hole, J15 through_hole, J16 through_hole, J17 through_hole, J18 through_hole, J19 through_hole, J20 through_hole, J21 through_hole, J5 through_hole, J6 through_hole, J7 through_hole, J8 through_hole, J9 through_hole, U1 scum3

Commit message: added LDOS
Parts:
- R4: symbol Device:R_Small_US -> scum3c-devboard-rescue:R_Small_US-Device
Changed lines of the file:
@@
 NoConn ~ 3500 1150
 $Comp
-L power:GND #PWR050
+L scum3c-devboard-rescue:GND-power #PWR050
 U 1 1 5F3D1F96
 P 2250 1700
@@
 $EndComp
 $Comp
-L power:GND #PWR052
+L scum3c-devboard-rescue:GND-power #PWR052
 U 1 1 5F3D443B
 P 2250 2600
@@
 $EndComp
 $Comp
-L power:GND #PWR054
+L scum3c-devboard-rescue:GND-power #PWR054
 U 1 1 5F3D4BFB
 P 2250 3500
@@
 $EndComp
 $Comp
-L power:GND #PWR055
+L scum3c-devboard-rescue:GND-power #PWR055
 U 1 1 5F3D5659
 P 2250 3950
@@
 $EndComp
 $Comp
-L power:GND #PWR056
+L scum3c-devboard-rescue:GND-power #PWR056
 U 1 1 5F3D5E43
 P 2250 4250
@@
 $EndComp
 $Comp
-L power:GND #PWR059
+L scum3c-devboard-rescue:GND-power #PWR059
 U 1 1 5F3DBD77
 P 3300 6050
@@
 $EndComp
 $Comp
-L power:GND #PWR063
+L scum3c-devboard-rescue:GND-power #PWR063
 U 1 1 5F3DC62E
 P 6300 6050
@@
 $EndComp
 $Comp
-L power:GND #PWR068
+L scum3c-devboard-rescue:GND-power #PWR068
 U 1 1 5F3DDBE9
 P 8000 4950
@@
 $EndComp
 $Comp
-L power:GND #PWR067
+L scum3c-devboard-rescue:GND-power #PWR067
 U 1 1 5F3DE6E7
 P 8000 4500
@@
 $EndComp
 $Comp
-L power:GND #PWR064
+L scum3c-devboard-rescue:GND-power #PWR064
 U 1 1 5F3DEB56
 P 8000 2850
@@
 $EndComp
 $Comp
-L Device:R_Small_US R4
+L scum3c-devboard-rescue:R_Small_US-Device R4
 U 1 1 61298275
 P 5000 900
