File: sulu-smartstake/scumsheet.kicad_sch (KiCad schematic)
At the start: 16 parts, among them J10 through_hole, J11 through_hole, J12 through_hole, J13 through_hole, J6 through_hole, J7 through_hole, J8 through_hole, J9 through_hole, U3 scum3

Commit message: Modify schematics after review
Parts:
- renumbered J7 to J10, J8 to J11, J9 to J12, J10 to J13, J11 to J14, J12 to J15, J13 to J16, J6 to J9
Changed lines of the file:
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@@
   (junction (at 238.76 60.96) (diameter 0) (color 0 0 0 0)
+  )
+  (junction (at 252.73 60.96) (diameter 0) (color 0 0 0 0)
   )
   (junction (at 132.08 17.78) (diameter 0) (color 0 0 0 0)
@@
     (stroke (width 0) (type default))
   )
+  (wire (pts (xy 209.55 102.87) (xy 212.09 102.87))
+    (stroke (width 0) (type default))
+  )
   (wire (pts (xy 209.55 60.96) (xy 238.76 60.96))
     (stroke (width 0) (type default))
@@
     (stroke (width 0) (type default))
   )
+  (wire (pts (xy 130.81 153.67) (xy 130.81 157.48))
+    (stroke (width 0) (type default))
+  )
   (wire (pts (xy 130.81 15.24) (xy 132.08 15.24))
     (stroke (width 0) (type default))
@@
     (stroke (width 0) (type default))
   )
+  (wire (pts (xy 252.73 59.69) (xy 252.73 60.96))
+    (stroke (width 0) (type default))
+  )
   (wire (pts (xy 50.8 130.81) (xy 63.5 130.81))
     (stroke (width 0) (type default))
   )
-  (wire (pts (xy 209.55 102.87) (xy 214.63 102.87))
-    (stroke (width 0) (type default))
-  )
   (wire (pts (xy 238.76 66.04) (xy 245.11 66.04))
     (stroke (width 0) (type default))
   )
-  (wire (pts (xy 130.81 153.67) (xy 130.81 158.75))
-    (stroke (width 0) (type default))
-  )
   (wire (pts (xy 209.55 99.06) (xy 214.63 99.06))
     (stroke (width 0) (type default))
   )
+  (wire (pts (xy 252.73 60.96) (xy 255.27 60.96))
+    (stroke (width 0) (type default))
+  )
   (wire (pts (xy 60.96 62.23) (xy 63.5 62.23))
     (stroke (width 0) (type default))
@@
     (stroke (width 0) (type default))
   )
-  (text_box "Important note: if the 1.1 V regulator is discarded, the BOOT_SOURCE_SEL pin must be tied to the VDDD_LDO_OUTPUT pin if 3WB should work.\n"
+  (text_box "Important note: If the 1.1 V regulator is discarded, the BOOT_SOURCE_SEL pin must be tied to the VDDD_LDO_OUTPUT pin for 3WB programming to work."
     (at 219.71 81.28 0) (size 41.91 10.16)
     (stroke (width 0) (type default))
@@
     (effects (font (size 1.27 1.27)) (justify left top))
   )
+  (label "VDDD_LDO_OUTPUT" (at 255.27 60.96 0) (fields_autoplaced)
+    (effects (font (size 1.27 1.27)) (justify left bottom))
+  )
+  (label "VDDD_LDO_OUTPUT" (at 212.09 102.87 0) (fields_autoplaced)
+    (effects (font (size 1.27 1.27)) (justify left bottom))
+  )
   (hierarchical_label "GPIO13" (shape bidirectional) (at 153.67 153.67 270) (fields_autoplaced)
     (effects (font (size 1.27 1.27)) (justify right))
   )
-  (hierarchical_label "+1.8V_REG" (shape input) (at 130.81 158.75 270) (fields_autoplaced)
+  (hierarchical_label "+1.8V_REG" (shape input) (at 130.81 157.48 270) (fields_autoplaced)
     (effects (font (size 1.27 1.27)) (justify right))
   )
@@
     (effects (font (size 1.27 1.27)) (justify left))
   )
-  (hierarchical_label "+1.1V_REG" (shape input) (at 214.63 102.87 0) (fields_autoplaced)
+  (hierarchical_label "+1.1V_REG" (shape input) (at 252.73 59.69 90) (fields_autoplaced)
     (effects (font (size 1.27 1.27)) (justify left))
   )
-  (hierarchical_label "+1.1V_REG" (shape input) (at 252.73 60.96 0) (fields_autoplaced)
-    (effects (font (size 1.27 1.27)) (justify left))
-  )
   (hierarchical_label "GPIO3" (shape bidirectional) (at 111.76 153.67 270) (fields_autoplaced)
     (effects (font (size 1.27 1.27)) (justify right))
@@
   (symbol (lib_id "draft1library:through_hole") (at 91.44 29.21 90) (unit 1)
     (in_bom yes) (on_board yes) (dnp no)
-    (property "Reference" "J9" (at 86.36 29.21 0)
+    (property "Reference" "J12" (at 86.36 29.21 0)
       (effects (font (size 1.27 1.27)) hide)
     )
@@
       (project "sulu_smartstake"
         (path "/def6aede-50f9-4865-b84d-079828465adb/1f92f92f-1391-4fc3-892c-7c652348c5b5"
-          (reference "J9") (unit 1)
+          (reference "J12") (unit 1)
         )
       )
@@
   (symbol (lib_id "draft1library:through_hole") (at 209.55 118.11 0) (unit 1)
     (in_bom yes) (on_board yes) (dnp no)
-    (property "Reference" "J12" (at 209.55 113.03 0)
+    (property "Reference" "J15" (at 209.55 113.03 0)
       (effects (font (size 1.27 1.27)) hide)
     )
@@
       (project "sulu_smartstake"
         (path "/def6aede-50f9-4865-b84d-079828465adb/1f92f92f-1391-4fc3-892c-7c652348c5b5"
-          (reference "J12") (unit 1)
+          (reference "J15") (unit 1)
         )
       )
@@
   (symbol (lib_id "draft1library:through_hole") (at 209.55 121.92 0) (unit 1)
     (in_bom yes) (on_board yes) (dnp no)
-    (property "Reference" "J13" (at 209.55 116.84 0)
+    (property "Reference" "J16" (at 209.55 116.84 0)
       (effects (font (size 1.27 1.27)) hide)
     )
@@
       (project "sulu_smartstake"
         (path "/def6aede-50f9-4865-b84d-079828465adb/1f92f92f-1391-4fc3-892c-7c652348c5b5"
-          (reference "J13") (unit 1)
+          (reference "J16") (unit 1)
         )
       )
@@
   )
   (symbol (lib_id "Device:C_Small") (at 245.11 63.5 0) (unit 1)
-    (in_bom yes) (on_board yes) (dnp no) (fields_autoplaced)
-    (property "Reference" "C11" (at 247.65 62.2362 0)
-      (effects (font (size 1.27 1.27)) (justify left))
-    )
-    (property "Value" "NP" (at 247.65 64.7762 0)
+    (in_bom yes) (on_board yes) (dnp no)
+    (property "Reference" "C11" (at 246.38 62.23 0)
+      (effects (font (size 1.27 1.27)) (justify left))
+    )
+    (property "Value" "NP" (at 246.38 64.77 0)
       (effects (font (size 1.27 1.27)) (justify left))
     )
@@
   (symbol (lib_id "draft1library:through_hole") (at 63.5 58.42 180) (unit 1)
     (in_bom yes) (on_board yes) (dnp no)
-    (property "Reference" "J7" (at 63.5 63.5 0)
+    (property "Reference" "J10" (at 63.5 63.5 0)
       (effects (font (size 1.27 1.27)) hide)
     )
@@
       (project "sulu_smartstake"
         (path "/def6aede-50f9-4865-b84d-079828465adb/1f92f92f-1391-4fc3-892c-7c652348c5b5"
-          (reference "J7") (unit 1)
+          (reference "J10") (unit 1)
         )
       )
@@
   (symbol (lib_id "draft1library:through_hole") (at 99.06 29.21 90) (unit 1)
     (in_bom yes) (on_board yes) (dnp no)
-    (property "Reference" "J10" (at 93.98 29.21 0)
+    (property "Reference" "J13" (at 93.98 29.21 0)
       (effects (font (size 1.27 1.27)) hide)
     )
@@
       (project "sulu_smartstake"
         (path "/def6aede-50f9-4865-b84d-079828465adb/1f92f92f-1391-4fc3-892c-7c652348c5b5"
-          (reference "J10") (unit 1)
+          (reference "J13") (unit 1)
         )
       )
@@
   (symbol (lib_id "draft1library:through_hole") (at 63.5 50.8 180) (unit 1)
     (in_bom yes) (on_board yes) (dnp no)
-    (property "Reference" "J6" (at 63.5 55.88 0)
+    (property "Reference" "J9" (at 63.5 55.88 0)
       (effects (font (size 1.27 1.27)) hide)
     )
@@
       (project "sulu_smartstake"
         (path "/def6aede-50f9-4865-b84d-079828465adb/1f92f92f-1391-4fc3-892c-7c652348c5b5"
-          (reference "J6") (unit 1)
+          (reference "J9") (unit 1)
         )
       )
@@
   (symbol (lib_id "draft1library:through_hole") (at 63.5 134.62 180) (unit 1)
     (in_bom yes) (on_board yes) (dnp no)
-    (property "Reference" "J8" (at 63.5 139.7 0)
+    (property "Reference" "J11" (at 63.5 139.7 0)
       (effects (font (size 1.27 1.27)) hide)
     )
@@
       (project "sulu_smartstake"
         (path "/def6aede-50f9-4865-b84d-079828465adb/1f92f92f-1391-4fc3-892c-7c652348c5b5"
-          (reference "J8") (unit 1)
+          (reference "J11") (unit 1)
         )
       )
@@
   (symbol (lib_id "draft1library:through_hole") (at 106.68 29.21 90) (unit 1)
     (in_bom yes) (on_board yes) (dnp no)
-    (property "Reference" "J11" (at 101.6 29.21 0)
+    (property "Reference" "J14" (at 101.6 29.21 0)
       (effects (font (size 1.27 1.27)) hide)
     )
@@
       (project "sulu_smartstake"
         (path "/def6aede-50f9-4865-b84d-079828465adb/1f92f92f-1391-4fc3-892c-7c652348c5b5"
-          (reference "J11") (unit 1)
-        )
-      )
+          (reference "J14") (unit 1)
+        )
+      )

Commit message: Finished layout after review
Parts:
- renumbered J9 to J10, J10 to J11, J11 to J12, J12 to J13, J13 to J14, J14 to J15, J15 to J16, J16 to J17
Changed lines of the file:
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@@
   (symbol (lib_id "draft1library:through_hole") (at 91.44 29.21 90) (unit 1)
     (in_bom yes) (on_board yes) (dnp no)
-    (property "Reference" "J12" (at 86.36 29.21 0)
+    (property "Reference" "J13" (at 86.36 29.21 0)
       (effects (font (size 1.27 1.27)) hide)
     )
@@
       (project "sulu_smartstake"
         (path "/def6aede-50f9-4865-b84d-079828465adb/1f92f92f-1391-4fc3-892c-7c652348c5b5"
-          (reference "J12") (unit 1)
+          (reference "J13") (unit 1)
         )
       )
@@
   (symbol (lib_id "draft1library:through_hole") (at 209.55 118.11 0) (unit 1)
     (in_bom yes) (on_board yes) (dnp no)
-    (property "Reference" "J15" (at 209.55 113.03 0)
+    (property "Reference" "J16" (at 209.55 113.03 0)
       (effects (font (size 1.27 1.27)) hide)
     )
@@
       (project "sulu_smartstake"
         (path "/def6aede-50f9-4865-b84d-079828465adb/1f92f92f-1391-4fc3-892c-7c652348c5b5"
-          (reference "J15") (unit 1)
+          (reference "J16") (unit 1)
         )
       )
@@
   (symbol (lib_id "draft1library:through_hole") (at 209.55 121.92 0) (unit 1)
     (in_bom yes) (on_board yes) (dnp no)
-    (property "Reference" "J16" (at 209.55 116.84 0)
+    (property "Reference" "J17" (at 209.55 116.84 0)
       (effects (font (size 1.27 1.27)) hide)
     )
@@
       (project "sulu_smartstake"
         (path "/def6aede-50f9-4865-b84d-079828465adb/1f92f92f-1391-4fc3-892c-7c652348c5b5"
-          (reference "J16") (unit 1)
+          (reference "J17") (unit 1)
         )
       )
@@
   (symbol (lib_id "draft1library:through_hole") (at 63.5 58.42 180) (unit 1)
     (in_bom yes) (on_board yes) (dnp no)
-    (property "Reference" "J10" (at 63.5 63.5 0)
+    (property "Reference" "J11" (at 63.5 63.5 0)
       (effects (font (size 1.27 1.27)) hide)
     )
@@
       (project "sulu_smartstake"
         (path "/def6aede-50f9-4865-b84d-079828465adb/1f92f92f-1391-4fc3-892c-7c652348c5b5"
-          (reference "J10") (unit 1)
+          (reference "J11") (unit 1)
         )
       )
@@
   (symbol (lib_id "draft1library:through_hole") (at 99.06 29.21 90) (unit 1)
     (in_bom yes) (on_board yes) (dnp no)
-    (property "Reference" "J13" (at 93.98 29.21 0)
+    (property "Reference" "J14" (at 93.98 29.21 0)
       (effects (font (size 1.27 1.27)) hide)
     )
@@
       (project "sulu_smartstake"
         (path "/def6aede-50f9-4865-b84d-079828465adb/1f92f92f-1391-4fc3-892c-7c652348c5b5"
-          (reference "J13") (unit 1)
+          (reference "J14") (unit 1)
         )
       )
@@
   (symbol (lib_id "draft1library:through_hole") (at 63.5 50.8 180) (unit 1)
     (in_bom yes) (on_board yes) (dnp no)
-    (property "Reference" "J9" (at 63.5 55.88 0)
+    (property "Reference" "J10" (at 63.5 55.88 0)
       (effects (font (size 1.27 1.27)) hide)
     )
@@
       (project "sulu_smartstake"
         (path "/def6aede-50f9-4865-b84d-079828465adb/1f92f92f-1391-4fc3-892c-7c652348c5b5"
-          (reference "J9") (unit 1)
+          (reference "J10") (unit 1)
         )
       )
@@
   (symbol (lib_id "draft1library:through_hole") (at 63.5 134.62 180) (unit 1)
     (in_bom yes) (on_board yes) (dnp no)
-    (property "Reference" "J11" (at 63.5 139.7 0)
+    (property "Reference" "J12" (at 63.5 139.7 0)
       (effects (font (size 1.27 1.27)) hide)
     )
@@
       (project "sulu_smartstake"
         (path "/def6aede-50f9-4865-b84d-079828465adb/1f92f92f-1391-4fc3-892c-7c652348c5b5"
-          (reference "J11") (unit 1)
+          (reference "J12") (unit 1)
         )
       )
@@
   (symbol (lib_id "draft1library:through_hole") (at 106.68 29.21 90) (unit 1)
     (in_bom yes) (on_board yes) (dnp no)
-    (property "Reference" "J14" (at 101.6 29.21 0)
+    (property "Reference" "J15" (at 101.6 29.21 0)
       (effects (font (size 1.27 1.27)) hide)
     )
@@
       (project "sulu_smartstake"
         (path "/def6aede-50f9-4865-b84d-079828465adb/1f92f92f-1391-4fc3-892c-7c652348c5b5"
-          (reference "J14") (unit 1)
-        )
-      )
+          (reference "J15") (unit 1)
+        )
+      )

Commit message: Final touches
Parts:
- added R3: 0 Ohm, Resistor_SMD:R_0402_1005Metric, symbol Device:R_US
- renumbered J11 to J10, J12 to J11, J13 to J12, J14 to J13, J15 to J14, J16 to J15, J17 to J16, J10 to J9
Connections:
- net +1.1V_REG: now also R3.2; no longer U3.61 (BOOT_SOURCE_SELECT)
- new net: R3.1, U3.61 (BOOT_SOURCE_SELECT)
Other:
- note added: "Look at bond diagram"
Changed lines of the file:
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@@
     (stroke (width 0) (type default))
   )
-  (wire (pts (xy 209.55 102.87) (xy 212.09 102.87))
+  (wire (pts (xy 209.55 102.87) (xy 228.6 102.87))
     (stroke (width 0) (type default))
   )
@@
   )
   (wire (pts (xy 238.76 60.96) (xy 245.11 60.96))
+    (stroke (width 0) (type default))
+  )
+  (wire (pts (xy 236.22 102.87) (xy 238.76 102.87))
     (stroke (width 0) (type default))
   )
@@
     (effects (font (size 1.27 1.27)) (justify left top))
   )
+  (text "Look at bond diagram" (at 76.2 19.05 0)
+    (effects (font (size 1.27 1.27)) (justify left bottom))
+  )
   (label "VDDD_LDO_OUTPUT" (at 255.27 60.96 0) (fields_autoplaced)
     (effects (font (size 1.27 1.27)) (justify left bottom))
   )
-  (label "VDDD_LDO_OUTPUT" (at 212.09 102.87 0) (fields_autoplaced)
+  (label "VDDD_LDO_OUTPUT" (at 238.76 102.87 0) (fields_autoplaced)
     (effects (font (size 1.27 1.27)) (justify left bottom))
   )
@@
   (symbol (lib_id "draft1library:through_hole") (at 91.44 29.21 90) (unit 1)
     (in_bom yes) (on_board yes) (dnp no)
-    (property "Reference" "J13" (at 86.36 29.21 0)
+    (property "Reference" "J12" (at 86.36 29.21 0)
       (effects (font (size 1.27 1.27)) hide)
     )
@@
       (project "sulu_smartstake"
         (path "/def6aede-50f9-4865-b84d-079828465adb/1f92f92f-1391-4fc3-892c-7c652348c5b5"
-          (reference "J13") (unit 1)
+          (reference "J12") (unit 1)
         )
       )
@@
   (symbol (lib_id "draft1library:through_hole") (at 209.55 118.11 0) (unit 1)
     (in_bom yes) (on_board yes) (dnp no)
-    (property "Reference" "J16" (at 209.55 113.03 0)
+    (property "Reference" "J15" (at 209.55 113.03 0)
       (effects (font (size 1.27 1.27)) hide)
     )
@@
       (project "sulu_smartstake"
         (path "/def6aede-50f9-4865-b84d-079828465adb/1f92f92f-1391-4fc3-892c-7c652348c5b5"
-          (reference "J16") (unit 1)
+          (reference "J15") (unit 1)
         )
       )
@@
   (symbol (lib_id "draft1library:through_hole") (at 209.55 121.92 0) (unit 1)
     (in_bom yes) (on_board yes) (dnp no)
-    (property "Reference" "J17" (at 209.55 116.84 0)
+    (property "Reference" "J16" (at 209.55 116.84 0)
       (effects (font (size 1.27 1.27)) hide)
     )
@@
       (project "sulu_smartstake"
         (path "/def6aede-50f9-4865-b84d-079828465adb/1f92f92f-1391-4fc3-892c-7c652348c5b5"
-          (reference "J17") (unit 1)
+          (reference "J16") (unit 1)
         )
       )
@@
   (symbol (lib_id "draft1library:through_hole") (at 63.5 58.42 180) (unit 1)
     (in_bom yes) (on_board yes) (dnp no)
-    (property "Reference" "J11" (at 63.5 63.5 0)
+    (property "Reference" "J10" (at 63.5 63.5 0)
       (effects (font (size 1.27 1.27)) hide)
     )
@@
       (project "sulu_smartstake"
         (path "/def6aede-50f9-4865-b84d-079828465adb/1f92f92f-1391-4fc3-892c-7c652348c5b5"
-          (reference "J11") (unit 1)
+          (reference "J10") (unit 1)
         )
       )
@@
   (symbol (lib_id "draft1library:through_hole") (at 99.06 29.21 90) (unit 1)
     (in_bom yes) (on_board yes) (dnp no)
-    (property "Reference" "J14" (at 93.98 29.21 0)
+    (property "Reference" "J13" (at 93.98 29.21 0)
       (effects (font (size 1.27 1.27)) hide)
     )
@@
       (project "sulu_smartstake"
         (path "/def6aede-50f9-4865-b84d-079828465adb/1f92f92f-1391-4fc3-892c-7c652348c5b5"
-          (reference "J14") (unit 1)
+          (reference "J13") (unit 1)
         )
       )
@@
   (symbol (lib_id "draft1library:through_hole") (at 63.5 50.8 180) (unit 1)
     (in_bom yes) (on_board yes) (dnp no)
-    (property "Reference" "J10" (at 63.5 55.88 0)
+    (property "Reference" "J9" (at 63.5 55.88 0)
       (effects (font (size 1.27 1.27)) hide)
     )
@@
       (project "sulu_smartstake"
         (path "/def6aede-50f9-4865-b84d-079828465adb/1f92f92f-1391-4fc3-892c-7c652348c5b5"
-          (reference "J10") (unit 1)
+          (reference "J9") (unit 1)
         )
       )
@@
     )
   )
+  (symbol (lib_id "Device:R_US") (at 232.41 102.87 90) (unit 1)
+    (in_bom yes) (on_board yes) (dnp no)
+    (property "Reference" "R3" (at 233.68 100.33 90)
+      (effects (font (size 1.27 1.27)) (justify left))
+    )
+    (property "Value" "0 Ohm" (at 234.95 105.41 90)
+      (effects (font (size 1.27 1.27)) (justify left))
+    )
+    (property "Footprint" "Resistor_SMD:R_0402_1005Metric" (at 232.664 101.854 90)
+      (effects (font (size 1.27 1.27)) hide)
+    )
+    (property "Datasheet" "~" (at 232.41 102.87 0)
+      (effects (font (size 1.27 1.27)) hide)
+    )
+    (pin "1")
+    (pin "2")
+    (instances
+      (project "sulu_smartstake"
+        (path "/def6aede-50f9-4865-b84d-079828465adb/1f92f92f-1391-4fc3-892c-7c652348c5b5"
+          (reference "R3") (unit 1)
+        )
+      )
+    )
+  )
   (symbol (lib_id "power:GND") (at 63.5 43.18 270) (unit 1)
     (in_bom yes) (on_board yes) (dnp no)
@@
   (symbol (lib_id "draft1library:through_hole") (at 63.5 134.62 180) (unit 1)
     (in_bom yes) (on_board yes) (dnp no)
-    (property "Reference" "J12" (at 63.5 139.7 0)
+    (property "Reference" "J11" (at 63.5 139.7 0)
       (effects (font (size 1.27 1.27)) hide)
     )
@@
       (project "sulu_smartstake"
         (path "/def6aede-50f9-4865-b84d-079828465adb/1f92f92f-1391-4fc3-892c-7c652348c5b5"
-          (reference "J12") (unit 1)
+          (reference "J11") (unit 1)
         )
       )
@@
   (symbol (lib_id "draft1library:through_hole") (at 106.68 29.21 90) (unit 1)
     (in_bom yes) (on_board yes) (dnp no)
-    (property "Reference" "J15" (at 101.6 29.21 0)
+    (property "Reference" "J14" (at 101.6 29.21 0)
       (effects (font (size 1.27 1.27)) hide)
     )
@@
       (project "sulu_smartstake"
         (path "/def6aede-50f9-4865-b84d-079828465adb/1f92f92f-1391-4fc3-892c-7c652348c5b5"
-          (reference "J15") (unit 1)
-        )
-      )
+          (reference "J14") (unit 1)
+        )
+      )
